File: PCB/PCB.kicad_sch (KiCad schematic)
At the start: 26 parts, among them U1 TPS54325, U2 TPS54294

Commit message: Finish sketch of power supply
Parts:
- added C17, C18: C, symbol Device:C
- added FB1: FerriteBead, symbol Device:FerriteBead
- added L3: L, symbol Device:L
- added R7, R8, R9: R, symbol Device:R
Connections:
- net GND: now also C10.2, C11.2, U2.4 (PGND1), U2.8 (GND), C17.2, C18.2, R8.2
- net at U2.10 (VFB2): now also R7.2, R8.1
- net at C9.2, U2.14 (SW2): now also L3.1
- new net: FB1.2, R9.1
- new net +3.3V: C17.1, C18.1, FB1.1, L3.2, R7.1, R9.2
Other:
- moved on the sheet: C1, C10, C11, C12, C13, C14, C15, C16, C2, C3, C4, C5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

Commit message: Add stuff
Parts:
- added C19: 1u, symbol Device:C
- C1: value C -> 3.3n
- C10, C13, C3: value C -> 10u
- C11, C12, C4, C5, C8, C9: value C -> 100n
- C14: value C -> 1u
- C15, C16, C17, C18, C6, C7: value C -> 22u
- C2: value C -> 100u
- L1, L2: value L -> 1.5u
- L3: value L -> 2.2u
- R1, R4: value R -> 100k
- R2: value R -> 6.81k
- R3, R6, R8: value R -> 22.1k
- R5: value R -> 30.1k
- R7: value R -> 73.2k
- R9: value R -> 1
Connections:
- net at C1.2, C2.2, C3.2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: now also C19.2
- net at R1.1, U1.3 (VREG5): now also C19.1
Other:
- moved on the sheet: C9

Commit message: Sketch
Parts:
- removed C1: 3.3n, symbol Device:C
- removed C10, C13, C3: 10u, symbol Device:C
- removed C11, C12, C4, C5, C8, C9: 100n, symbol Device:C
- removed C14, C19: 1u, symbol Device:C
- removed C15, C16, C17, C18, C6, C7: 22u, symbol Device:C
- removed C2: 100u, symbol Device:C
- removed FB1: FerriteBead, symbol Device:FerriteBead
- removed L1, L2: 1.5u, symbol Device:L
- removed L3: 2.2u, symbol Device:L
- removed R1, R4: 100k, symbol Device:R
- removed R2: 6.81k, symbol Device:R
- removed R3, R6, R8: 22.1k, symbol Device:R
- removed R5: 30.1k, symbol Device:R
- removed R7: 73.2k, symbol Device:R
- removed R9: 1, symbol Device:R
- removed U1: TPS54325, symbol Components_Library:TPS54325
- removed U2: TPS54294, symbol Components_Library:TPS54294
Other:
- added sheet microcontroller_unit (mcu.kicad_sch)
- added sheet power_supply (power_supply.kicad_sch)

Commit message: Added FPGA
Other:
- added sheet FPGA (fpga.kicad_sch)
Changed lines of the file:
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@@
+    )
+  )
+  (sheet (at 120.65 85.09) (size 33.02 26.67) (fields_autoplaced)
+    (stroke (width 0.1524) (type solid))
+    (fill (color 0 0 0 0.0000))
+    (property "Sheetname" "FPGA" (at 120.65 84.3784 0)
+      (effects (font (size 1.27 1.27)) (justify left bottom))
+    )
+    (property "Sheetfile" "fpga.kicad_sch" (at 120.65 112.3446 0)
+      (effects (font (size 1.27 1.27)) (justify left top))
+    )
+    (instances
+      (project "PCB"
+        (path "/aa113cd6-c3ac-4890-9a84-1ea195994408" (page "4"))
+      )
     )
   )

Commit message: Work
Other:
- sheet microcontroller_unit ports: added 5V; removed none
- sheet power_supply ports: added 5V; removed none
Changed lines of the file:
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@@
 (kicad_sch (version 20230121) (generator eeschema)
   (paper "A4")
-  (sheet (at 165.1 43.18) (size 33.02 27.94) (fields_autoplaced)
+  (wire (pts (xy 99.06 55.88) (xy 127 55.88))
+    (stroke (width 0) (type default))
+  )
+  (sheet (at 127 41.91) (size 33.02 27.94) (fields_autoplaced)
     (stroke (width 0.1524) (type solid))
     (fill (color 0 0 0 0.0000))
-    (property "Sheetname" "microcontroller_unit" (at 165.1 42.4684 0)
+    (property "Sheetname" "microcontroller_unit" (at 127 41.1984 0)
       (effects (font (size 1.27 1.27)) (justify left bottom))
     )
-    (property "Sheetfile" "mcu.kicad_sch" (at 165.1 71.7046 0)
+    (property "Sheetfile" "mcu.kicad_sch" (at 127 70.4346 0)
       (effects (font (size 1.27 1.27)) (justify left top))
+    )
+    (pin "5V" input (at 127 55.88 180)
+      (effects (font (size 1.27 1.27)) (justify left))
     )
     (instances
@@
       (effects (font (size 1.27 1.27)) (justify left top))
     )
+    (pin "5V" input (at 99.06 55.88 0)
+      (effects (font (size 1.27 1.27)) (justify right))
+    )
     (instances
       (project "PCB"
@@
     )
   )
-  (sheet (at 120.65 85.09) (size 33.02 26.67) (fields_autoplaced)
+  (sheet (at 120.65 86.36) (size 35.56 25.4) (fields_autoplaced)
     (stroke (width 0.1524) (type solid))
     (fill (color 0 0 0 0.0000))
-    (property "Sheetname" "FPGA" (at 120.65 84.3784 0)
+    (property "Sheetname" "FPGA" (at 120.65 85.6484 0)
       (effects (font (size 1.27 1.27)) (justify left bottom))
     )

Commit message: more work
Other:
- sheet FPGA ports: added CLK, CS, MISO, MOSI, done, program_b; removed none
- sheet microcontroller_unit ports: added 5V_IN, CLK, CS, MISO, MOSI; removed 5V
- sheet power_supply ports: added 5V_OUT; removed 5V
Changed lines of the file:
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@@
 (kicad_sch (version 20230121) (generator eeschema)
   (paper "A4")
-  (wire (pts (xy 99.06 55.88) (xy 127 55.88))
+  (wire (pts (xy 137.16 69.85) (xy 137.16 86.36))
+    (stroke (width 0) (type default))
+  )
+  (wire (pts (xy 114.3 54.61) (xy 127 54.61))
+    (stroke (width 0) (type default))
+  )
+  (wire (pts (xy 133.35 69.85) (xy 133.35 86.36))
+    (stroke (width 0) (type default))
+  )
+  (wire (pts (xy 130.81 69.85) (xy 130.81 86.36))
+    (stroke (width 0) (type default))
+  )
+  (wire (pts (xy 140.97 69.85) (xy 140.97 86.36))
     (stroke (width 0) (type default))
   )
@@
       (effects (font (size 1.27 1.27)) (justify left top))
     )
-    (pin "5V" input (at 127 55.88 180)
+    (pin "5V_IN" input (at 127 54.61 180)
+      (effects (font (size 1.27 1.27)) (justify left))
+    )
+    (pin "MISO" input (at 130.81 69.85 270)
+      (effects (font (size 1.27 1.27)) (justify left))
+    )
+    (pin "MOSI" input (at 133.35 69.85 270)
+      (effects (font (size 1.27 1.27)) (justify left))
+    )
+    (pin "CS" input (at 137.16 69.85 270)
+      (effects (font (size 1.27 1.27)) (justify left))
+    )
+    (pin "CLK" input (at 140.97 69.85 270)
       (effects (font (size 1.27 1.27)) (justify left))
     )
@@
     )
   )
-  (sheet (at 76.2 46.99) (size 22.86 19.05) (fields_autoplaced)
+  (sheet (at 91.44 45.72) (size 22.86 19.05) (fields_autoplaced)
     (stroke (width 0.1524) (type solid))
     (fill (color 0 0 0 0.0000))
-    (property "Sheetname" "power_supply" (at 76.2 46.2784 0)
+    (property "Sheetname" "power_supply" (at 91.44 45.0084 0)
       (effects (font (size 1.27 1.27)) (justify left bottom))
     )
-    (property "Sheetfile" "power_supply.kicad_sch" (at 76.2 66.6246 0)
+    (property "Sheetfile" "power_supply.kicad_sch" (at 91.44 65.3546 0)
       (effects (font (size 1.27 1.27)) (justify left top))
     )
-    (pin "5V" input (at 99.06 55.88 0)
+    (pin "5V_OUT" input (at 114.3 54.61 0)
       (effects (font (size 1.27 1.27)) (justify right))
     )
@@
       (effects (font (size 1.27 1.27)) (justify left top))
     )
+    (pin "done" input (at 149.86 86.36 90)
+      (effects (font (size 1.27 1.27)) (justify right))
+    )
+    (pin "program_b" input (at 147.32 86.36 90)
+      (effects (font (size 1.27 1.27)) (justify right))
+    )
+    (pin "CLK" input (at 140.97 86.36 90)
+      (effects (font (size 1.27 1.27)) (justify right))
+    )
+    (pin "MISO" input (at 130.81 86.36 90)
+      (effects (font (size 1.27 1.27)) (justify right))
+    )
+    (pin "CS" input (at 137.16 86.36 90)
+      (effects (font (size 1.27 1.27)) (justify right))
+    )
+    (pin "MOSI" input (at 133.35 86.36 90)
+      (effects (font (size 1.27 1.27)) (justify right))
+    )
     (instances

Commit message: work
Other:
- sheet FPGA ports: added GPIO0, GPIO1, GPIO2, GPIO3, GPIO4, GPIO5, GPIO6, GPIO7; removed none
- sheet microcontroller_unit ports: added GPIO0, GPIO1, GPIO2, GPIO3, GPIO4, GPIO5, GPIO6, GPIO7; removed none
Changed lines of the file:
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@@
 (kicad_sch (version 20230121) (generator eeschema)
   (paper "A4")
+  (wire (pts (xy 156.21 96.52) (xy 161.29 96.52))
+    (stroke (width 0) (type default))
+  )
+  (wire (pts (xy 171.45 54.61) (xy 171.45 106.68))
+    (stroke (width 0) (type default))
+  )
+  (wire (pts (xy 163.83 62.23) (xy 163.83 99.06))
+    (stroke (width 0) (type default))
+  )
   (wire (pts (xy 137.16 69.85) (xy 137.16 86.36))
+    (stroke (width 0) (type default))
+  )
+  (wire (pts (xy 166.37 101.6) (xy 156.21 101.6))
+    (stroke (width 0) (type default))
+  )
+  (wire (pts (xy 166.37 59.69) (xy 160.02 59.69))
     (stroke (width 0) (type default))
   )
@@
     (stroke (width 0) (type default))
   )
+  (wire (pts (xy 168.91 57.15) (xy 160.02 57.15))
+    (stroke (width 0) (type default))
+  )
   (wire (pts (xy 133.35 69.85) (xy 133.35 86.36))
+    (stroke (width 0) (type default))
+  )
+  (wire (pts (xy 146.05 69.85) (xy 146.05 86.36))
+    (stroke (width 0) (type default))
+  )
+  (wire (pts (xy 156.21 99.06) (xy 163.83 99.06))
+    (stroke (width 0) (type default))
+  )
+  (wire (pts (xy 161.29 64.77) (xy 161.29 96.52))
+    (stroke (width 0) (type default))
+  )
+  (wire (pts (xy 161.29 64.77) (xy 160.02 64.77))
+    (stroke (width 0) (type default))
+  )
+  (wire (pts (xy 166.37 59.69) (xy 166.37 101.6))
+    (stroke (width 0) (type default))
+  )
+  (wire (pts (xy 156.21 104.14) (xy 168.91 104.14))
+    (stroke (width 0) (type default))
+  )
+  (wire (pts (xy 160.02 62.23) (xy 163.83 62.23))
+    (stroke (width 0) (type default))
+  )
+  (wire (pts (xy 168.91 57.15) (xy 168.91 104.14))
+    (stroke (width 0) (type default))
+  )
+  (wire (pts (xy 171.45 54.61) (xy 160.02 54.61))
+    (stroke (width 0) (type default))
+  )
+  (wire (pts (xy 148.59 69.85) (xy 148.59 86.36))
+    (stroke (width 0) (type default))
+  )
+  (wire (pts (xy 156.21 106.68) (xy 171.45 106.68))
     (stroke (width 0) (type default))
   )
@@
     (stroke (width 0) (type default))
   )
-  (sheet (at 127 41.91) (size 33.02 27.94) (fields_autoplaced)
+  (wire (pts (xy 151.13 69.85) (xy 151.13 86.36))
+    (stroke (width 0) (type default))
+  )
+  (sheet (at 127 41.91) (size 33.02 27.94)
     (stroke (width 0.1524) (type solid))
     (fill (color 0 0 0 0.0000))
@@
       (effects (font (size 1.27 1.27)) (justify left bottom))
     )
-    (property "Sheetfile" "mcu.kicad_sch" (at 127 70.4346 0)
+    (property "Sheetfile" "mcu.kicad_sch" (at 146.05 74.93 0)
       (effects (font (size 1.27 1.27)) (justify left top))
     )
@@
     )
     (pin "CLK" input (at 140.97 69.85 270)
+      (effects (font (size 1.27 1.27)) (justify left))
+    )
+    (pin "GPIO2" input (at 160.02 59.69 0)
+      (effects (font (size 1.27 1.27)) (justify right))
+    )
+    (pin "GPIO3" input (at 160.02 62.23 0)
+      (effects (font (size 1.27 1.27)) (justify right))
+    )
+    (pin "GPIO0" input (at 160.02 54.61 0)
+      (effects (font (size 1.27 1.27)) (justify right))
+    )
+    (pin "GPIO1" input (at 160.02 57.15 0)
+      (effects (font (size 1.27 1.27)) (justify right))
+    )
+    (pin "GPIO4" input (at 160.02 64.77 0)
+      (effects (font (size 1.27 1.27)) (justify right))
+    )
+    (pin "GPIO5" input (at 151.13 69.85 270)
+      (effects (font (size 1.27 1.27)) (justify left))
+    )
+    (pin "GPIO6" input (at 148.59 69.85 270)
+      (effects (font (size 1.27 1.27)) (justify left))
+    )
+    (pin "GPIO7" input (at 146.05 69.85 270)
       (effects (font (size 1.27 1.27)) (justify left))
     )
@@
       (effects (font (size 1.27 1.27)) (justify left top))
     )
-    (pin "done" input (at 149.86 86.36 90)
-      (effects (font (size 1.27 1.27)) (justify right))
+    (pin "done" input (at 120.65 100.33 180)
+      (effects (font (size 1.27 1.27)) (justify left))
     )
-    (pin "program_b" input (at 147.32 86.36 90)
-      (effects (font (size 1.27 1.27)) (justify right))
+    (pin "program_b" input (at 120.65 96.52 180)
+      (effects (font (size 1.27 1.27)) (justify left))
     )
     (pin "CLK" input (at 140.97 86.36 90)
@@
       (effects (font (size 1.27 1.27)) (justify right))
     )
+    (pin "GPIO0" input (at 156.21 106.68 0)
+      (effects (font (size 1.27 1.27)) (justify right))
+    )
+    (pin "GPIO1" input (at 156.21 104.14 0)
+      (effects (font (size 1.27 1.27)) (justify right))
+    )
+    (pin "GPIO2" input (at 156.21 101.6 0)
+      (effects (font (size 1.27 1.27)) (justify right))
+    )
+    (pin "GPIO3" input (at 156.21 99.06 0)
+      (effects (font (size 1.27 1.27)) (justify right))
+    )
+    (pin "GPIO5" input (at 151.13 86.36 90)
+      (effects (font (size 1.27 1.27)) (justify right))
+    )
+    (pin "GPIO7" input (at 146.05 86.36 90)
+      (effects (font (size 1.27 1.27)) (justify right))
+    )
+    (pin "GPIO4" input (at 156.21 96.52 0)
+      (effects (font (size 1.27 1.27)) (justify right))
+    )
+    (pin "GPIO6" input (at 148.59 86.36 90)
+      (effects (font (size 1.27 1.27)) (justify right))
+    )
