File: PCB/PCB.kicad_sch (KiCad schematic)
At the start: 0 parts

Commit message: Add
Parts:
- added C24, C25, C26, C27, C28, C29, C43, C44, C50, C51, C61, C62, C68, C69, C75, C76, C82, C83: 4.7u, symbol Device:C
- added C30, C31, C32, C33, C34, C35, C36, C38, C40, C41, C45, C46, C47, C52, C53, C54, C55, C56, C58, C59, C60, C64, C65, C66, C67, C71, C72, C73, C74, C78, C79, C80, C81: 470n, symbol Device:C
- added C37: 330u, symbol Device:C
- added C39: 100u, symbol Device:C
- added C42, C48, C49, C63, C70, C77, C84: 47u, symbol Device:C
Connections:
- new net +1V0: C24.1, C25.1, C26.1, C27.1, C28.1, C29.1, C30.1, C31.1, C32.1, C33.1, C34.1, C35.1, C36.1, C37.1, C38.1, C39.1, C40.1, C41.1
- new net +1V8: C42.1, C43.1, C44.1, C45.1, C46.1, C47.1
- new net +3.3V: C48.1, C49.1, C50.1, C51.1, C52.1, C53.1, C54.1, C55.1, C56.1, C58.1, C59.1, C60.1, C61.1, C62.1, C63.1, C64.1, C65.1, C66.1, C67.1, C68.1, C69.1, C70.1, C71.1, C72.1, C73.1, C74.1, C75.1, C76.1, C77.1, C78.1, C79.1, C80.1, C81.1, C82.1, C83.1, C84.1
- new net GND: C24.2, C25.2, C26.2, C27.2, C28.2, C29.2, C30.2, C31.2, C32.2, C33.2, C34.2, C35.2, C36.2, C37.2, C38.2, C39.2, C40.2, C41.2, C42.2, C43.2, C44.2, C45.2, C46.2, C47.2, C48.2, C49.2, C50.2, C51.2, C52.2, C53.2, C54.2, C55.2, C56.2, C58.2, C59.2, C60.2, C61.2, C62.2, C63.2, C64.2, C65.2, C66.2, C67.2, C68.2, C69.2, C70.2, C71.2, C72.2, C73.2, C74.2, C75.2, C76.2, C77.2, C78.2, C79.2, C80.2, C81.2, C82.2, C83.2, C84.2
Other:
- added sheet VGA (vga.kicad_sch)
- sheet FPGA ports: added BLUE0, BLUE1, BLUE2, BLUE3, BLUE4, GREEN0, GREEN1, GREEN2, GREEN3, GREEN4, HSYNC, RED0, RED1, RED2, RED3, RED4, VSYNC; removed none

Commit message: Footprints
Parts:
- C24, C25, C26, C27, C28, C29, C30, C31, C32, C33, C34, C35, C36, C37, C38, C39, C40, C41, C42, C43, C44, C45, C46, C47, C48, C49, C50, C51, C52, C53, C54, C55, C56, C58, C59, C60, C61, C62, C63, C64, C65, C66, C67, C68, C69, C70, C71, C72, C73, C74, C75, C76, C77, C78, C79, C80, C81, C82, C83, C84: footprint (none) -> Capacitor_SMD:C_0805_2012Metric_Pad1.18x1.45mm_HandSolder
Connections:
- no-connect marks 0 -> 2

Commit message: schematic fixes
Connections:
- no-connect marks 2 -> 0
Other:
- sheet microcontroller_unit ports: added done, program_b; removed none
Changed lines of the file:
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@@
   (junction (at 54.61 119.38) (diameter 0) (color 0 0 0 0)
   )
-  (no_connect (at 92.71 96.52))
-  (no_connect (at 92.71 100.33))
   (wire (pts (xy 156.21 96.52) (xy 161.29 96.52))
     (stroke (width 0) (type default))
@@
     (stroke (width 0) (type default))
   )
+  (wire (pts (xy 89.535 96.52) (xy 92.71 96.52))
+    (stroke (width 0) (type default))
+  )
   (wire (pts (xy 191.77 96.52) (xy 191.77 102.87))
     (stroke (width 0) (type default))
@@
     (stroke (width 0) (type default))
   )
+  (wire (pts (xy 120.015 61.595) (xy 127 61.595))
+    (stroke (width 0) (type default))
+  )
   (wire (pts (xy 27.94 104.14) (xy 27.94 111.76))
     (stroke (width 0) (type default))
@@
     (stroke (width 0) (type default))
   )
+  (wire (pts (xy 120.015 82.55) (xy 89.535 82.55))
+    (stroke (width 0) (type default))
+  )
   (wire (pts (xy 62.23 104.14) (xy 62.23 111.76))
     (stroke (width 0) (type default))
@@
     (stroke (width 0) (type default))
   )
+  (wire (pts (xy 92.71 100.33) (xy 86.36 100.33))
+    (stroke (width 0) (type default))
+  )
   (wire (pts (xy 114.3 121.92) (xy 114.3 127))
     (stroke (width 0) (type default))
@@
     (stroke (width 0) (type default))
   )
+  (wire (pts (xy 116.84 78.74) (xy 116.84 58.42))
+    (stroke (width 0) (type default))
+  )
   (wire (pts (xy 246.38 57.15) (xy 246.38 49.53))
     (stroke (width 0) (type default))
@@
     (stroke (width 0) (type default))
   )
+  (wire (pts (xy 116.84 58.42) (xy 127 58.42))
+    (stroke (width 0) (type default))
+  )
   (wire (pts (xy 40.64 81.28) (xy 40.64 88.9))
     (stroke (width 0) (type default))
@@
     (stroke (width 0) (type default))
   )
+  (wire (pts (xy 86.36 78.74) (xy 116.84 78.74))
+    (stroke (width 0) (type default))
+  )
   (wire (pts (xy 68.58 96.52) (xy 68.58 104.14))
     (stroke (width 0) (type default))
@@
     (stroke (width 0) (type default))
   )
+  (wire (pts (xy 86.36 100.33) (xy 86.36 78.74))
+    (stroke (width 0) (type default))
+  )
   (wire (pts (xy 68.58 73.66) (xy 68.58 81.28))
     (stroke (width 0) (type default))
@@
     (stroke (width 0) (type default))
   )
+  (wire (pts (xy 120.015 61.595) (xy 120.015 82.55))
+    (stroke (width 0) (type default))
+  )
   (wire (pts (xy 76.2 176.53) (xy 76.2 185.42))
     (stroke (width 0) (type default))
@@
   )
   (wire (pts (xy 27.94 81.28) (xy 27.94 88.9))
+    (stroke (width 0) (type default))
+  )
+  (wire (pts (xy 89.535 82.55) (xy 89.535 96.52))
     (stroke (width 0) (type default))
   )
@@
       (effects (font (size 1.27 1.27)) (justify left))
     )
+    (pin "program_b" input (at 127 61.595 180)
+      (effects (font (size 1.27 1.27)) (justify left))
+    )
+    (pin "done" input (at 127 58.42 180)
+      (effects (font (size 1.27 1.27)) (justify left))
+    )

Commit message: updates
Parts:
- C37: footprint Capacitor_SMD:C_0805_2012Metric_Pad1.18x1.45mm_HandSolder -> Capacitor_SMD:C_1206_3216Metric_Pad1.33x1.80mm_HandSolder
Changed lines of the file:
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@@
       (effects (font (size 1.27 1.27)) (justify left))
     )
-    (property "Footprint" "Capacitor_SMD:C_0805_2012Metric_Pad1.18x1.45mm_HandSolder" (at 199.39 114.6048 0)
+    (property "Footprint" "Capacitor_SMD:C_1206_3216Metric_Pad1.33x1.80mm_HandSolder" (at 199.39 114.6048 0)
       (effects (font (size 1.27 1.27)) hide)
     )
