File: PCB/fpga.kicad_sch (KiCad schematic)
At the start: 47 parts, among them IC1 S25FL256LAGMFI003, J1 0878311420, U4 XC7A100T-FTG256, U5 IS62C1024AL-35QLI-TR, Y2 ECS-3953M-400-BN-TR

Commit message: more work
Connections:
- net MOSI: now reaches U4.A8 (IO_L2P_T0_AD8P_15)
- net CS: now reaches U4.C8 (IO_L1P_T0_AD0P_15)
- net MISO: now reaches U4.C9 (IO_L1N_T0_AD0N_15)
- net CLK: now reaches U4.D10 (IO_0_15)
Changed lines of the file:
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@@
+    (stroke (width 0) (type default))
+  )
+  (wire (pts (xy 167.64 46.99) (xy 171.45 46.99))
     (stroke (width 0) (type default))
   )
@@
     (stroke (width 0) (type default))
   )
+  (wire (pts (xy 167.64 41.91) (xy 171.45 41.91))
+    (stroke (width 0) (type default))
+  )
   (wire (pts (xy 280.67 36.83) (xy 275.59 36.83))
     (stroke (width 0) (type default))
@@
     (stroke (width 0) (type default))
   )
+  (wire (pts (xy 167.64 44.45) (xy 171.45 44.45))
+    (stroke (width 0) (type default))
+  )
   (wire (pts (xy 280.67 19.05) (xy 280.67 21.59))
     (stroke (width 0) (type default))
@@
     (stroke (width 0) (type default))
   )
+  (wire (pts (xy 167.64 49.53) (xy 171.45 49.53))
+    (stroke (width 0) (type default))
+  )
   (wire (pts (xy 280.67 74.93) (xy 280.67 77.47))
     (stroke (width 0) (type default))
@@
     (stroke (width 0) (type default))
   )
+  (label "SPI to MCU" (at 180.34 45.72 0) (fields_autoplaced)
+    (effects (font (size 1.27 1.27)) (justify left bottom))
+  )
+  (hierarchical_label "CLK" (shape input) (at 171.45 41.91 0) (fields_autoplaced)
+    (effects (font (size 1.27 1.27)) (justify left))
+  )
+  (hierarchical_label "MOSI" (shape input) (at 171.45 49.53 0) (fields_autoplaced)
+    (effects (font (size 1.27 1.27)) (justify left))
+  )
+  (hierarchical_label "CS" (shape input) (at 171.45 44.45 0) (fields_autoplaced)
+    (effects (font (size 1.27 1.27)) (justify left))
+  )
+  (hierarchical_label "MISO" (shape input) (at 171.45 46.99 0) (fields_autoplaced)
+    (effects (font (size 1.27 1.27)) (justify left))
+  )
   (hierarchical_label "done" (shape input) (at 54.61 95.885 90) (fields_autoplaced)

Commit message: work
Parts:
- added C56, C58, C59, C60, C64, C65, C66, C67, C71, C72, C73, C74, C78, C79, C80, C81: 470n, symbol Device:C
- added C61, C62, C68, C69, C75, C76, C82, C83: 4.7u, symbol Device:C
- added C63, C70, C77, C84: 47u, symbol Device:C
- added J4: 62684-402100ALF, 62684402100ALF, symbol 62684-402100ALF:62684-402100ALF
Connections:
- net +3.3V: now also U4.A6 (VCCO_35), U4.B3 (VCCO_35), U4.D7 (VCCO_35), U4.E4 (VCCO_35), U4.F1 (VCCO_35), U4.J2 (VCCO_35), U4.M3 (VCCO_34), U4.R4 (VCCO_34), U4.T1 (VCCO_34), C56.1, C58.1, C59.1, C60.1, C61.1, C62.1, C63.1, C64.1, C65.1, C66.1, C67.1, C68.1, C69.1, C70.1, C71.1, C72.1, C73.1, C74.1, C75.1, C76.1, C77.1, C78.1, C79.1, C80.1, C81.1, C82.1, C83.1, C84.1
- net GND: now also U4.A13 (IO_L7P_T1_AD2P_15), U4.A14 (IO_L7N_T1_AD2N_15), U4.A15 (IO_L9N_T1_DQS_AD3N_15), U4.A3 (IO_L4N_T0_35), U4.A4 (IO_L3N_T0_DQS_AD5N_35), U4.A5 (IO_L3P_T0_DQS_AD5P_35), U4.A7 (IO_L1N_T0_AD4N_35), U4.B14 (IO_L8N_T1_AD10N_15), U4.B15 (IO_L9P_T1_DQS_AD3P_15), U4.B16 (IO_L10N_T1_AD11N_15), U4.B4 (IO_L4P_T0_35), U4.B5 (IO_L2N_T0_AD12N_35), U4.B6 (IO_L2P_T0_AD12P_35), U4.B7 (IO_L1P_T0_AD4P_35), U4.C14 (IO_L8P_T1_AD10P_15), U4.C16 (IO_L10P_T1_AD11P_15), U4.C7 (IO_L5P_T0_AD13P_35), U4.D9 (IO_L6N_T0_VREF_15), U4.E6 (IO_0_35), U4.K13 (IO_L5P_T0_D06_14), U4.L13 (IO_L5N_T0_D07_14), U4.L14 (IO_L4P_T0_D04_14), U4.L4 (IO_L1P_T0_34), U4.L5 (IO_0_34), U4.M1 (IO_L2N_T0_34), U4.M12 (IO_L6N_T0_D08_VREF_14), U4.M14 (IO_L4N_T0_D05_14), U4.M15 (IO_L3N_T0_DQS_EMCCLK_14), U4.M16 (IO_L7P_T1_D09_14), U4.M2 (IO_L2P_T0_34), U4.M4 (IO_L1N_T0_34), U4.M5 (IO_L6P_T0_34), U4.M6 (IO_L19P_T3_A10_D26_14), U4.N1 (IO_L4P_T0_34), U4.N12 (IO_L13N_T2_MRCC_14), U4.N13 (IO_L11P_T1_SRCC_14), U4.N14 (IO_L12P_T1_MRCC_14), U4.N16 (IO_L7N_T1_D10_14), U4.N2 (IO_L3N_T0_DQS_34), U4.N3 (IO_L3P_T0_DQS_34), U4.N4 (IO_L6N_T0_VREF_34), U4.N6 (IO_L19N_T3_A09_D25_VREF_14), U4.N9 (IO_L18P_T2_A12_D28_14), U4.P1 (IO_L4N_T0_34), U4.P10 (IO_L14P_T2_SRCC_14), U4.P11 (IO_L14N_T2_SRCC_14), U4.P13 (IO_L11N_T1_SRCC_14), U4.P14 (IO_L12N_T1_MRCC_14), U4.P15 (IO_L8P_T1_D11_14), U4.P16 (IO_L8N_T1_D12_14), U4.P3 (IO_L5N_T0_34), U4.P4 (IO_L5P_T0_34), U4.P5 (IO_L10P_T1_34), U4.P6 (IO_25_14), U4.P8 (IO_L20P_T3_A08_D24_14), U4.P9 (IO_L18N_T2_A11_D27_14), U4.R1 (IO_L7N_T1_34), U4.R10 (IO_L17P_T2_A14_D30_14), U4.R11 (IO_L17N_T2_A13_D29_14), U4.R12 (IO_L15P_T2_DQS_RDWR_B_14), U4.R13 (IO_L16P_T2_CSI_B_14), U4.R15 (IO_L9P_T1_DQS_14), U4.R16 (IO_L9N_T1_DQS_D13_14), U4.R2 (IO_L7P_T1_34), U4.R3 (IO_L8P_T1_34), U4.R5 (IO_L23P_T3_A03_D19_14), U4.R6 (IO_L24P_T3_A01_D17_14), U4.R7 (IO_L24N_T3_A00_D16_14), U4.R8 (IO_L20N_T3_A07_D23_14), U4.T10 (IO_L22N_T3_A04_D20_14), U4.T12 (IO_L15N_T2_DQS_DOUT_CSO_B_14), U4.T13 (IO_L16N_T2_A15_D31_14), U4.T14 (IO_L10P_T1_D14_14), U4.T15 (IO_L10N_T1_D15_14), U4.T2 (IO_L8N_T1_34), U4.T3 (IO_L9N_T1_DQS_34), U4.T4 (IO_L9P_T1_DQS_34), U4.T5 (IO_L23N_T3_A02_D18_14), U4.T7 (IO_L21P_T3_DQS_14), U4.T8 (IO_L21N_T3_DQS_A06_D22_14), U4.T9 (IO_L22P_T3_A05_D21_14), C56.2, C58.2, C59.2, C60.2, C61.2, C62.2, C63.2, C64.2, C65.2, C66.2, C67.2, C68.2, C69.2, C70.2, C71.2, C72.2, C73.2, C74.2, C75.2, C76.2, C77.2, C78.2, C79.2, C80.2, C81.2, C82.2, C83.2, C84.2, J4.MH1, J4.MH2
- net GPIO2: now reaches U4.A10 (IO_L3N_T0_DQS_AD1N_15)
- net GPIO6: now reaches U4.A12 (IO_L5N_T0_AD9N_15)
- net GPIO0: now reaches U4.A9 (IO_L2N_T0_AD8N_15)
- net GPIO3: now reaches U4.B10 (IO_L4P_T0_15)
- net GPIO4: now reaches U4.B11 (IO_L4N_T0_15)
- net GPIO5: now reaches U4.B12 (IO_L5P_T0_AD9P_15)
- net GPIO1: now reaches U4.B9 (IO_L3P_T0_DQS_AD1P_15)
- net GPIO7: now reaches U4.D8 (IO_L6P_T0_15)
- net at U4.K16 (IO_L2N_T0_D03_14): now also IC1.1 (IO3_/_RESET#), R15.2
- net at U4.A2 (IO_L8N_T1_AD14N_35): now also J4.7
- net at U4.B1 (IO_L9N_T1_DQS_AD7N_35): now also J4.9
- net at U4.B2 (IO_L8P_T1_AD14P_35): now also J4.6
- net at U4.C1 (IO_L9P_T1_DQS_AD7P_35): now also J4.8
- net at U4.C2 (IO_L7N_T1_AD6N_35): now also J4.5
- net at U4.C3 (IO_L7P_T1_AD6P_35): now also J4.4
- net at U4.C4 (IO_L12N_T1_MRCC_35): now also J4.15
- net at U4.C6 (IO_L5N_T0_AD13N_35): now also J4.1
- net at U4.D1 (IO_L10N_T1_AD15N_35): now also J4.11
- net at U4.D3 (IO_L11N_T1_SRCC_35): now also J4.13
- net at U4.D4 (IO_L12P_T1_MRCC_35): now also J4.14
- net at U4.D5 (IO_L6N_T0_VREF_35): now also J4.3
- net at U4.D6 (IO_L6P_T0_35): now also J4.2
- net at U4.E1 (IO_L15N_T2_DQS_35): now also J4.21
- net at U4.E2 (IO_L10P_T1_AD15P_35): now also J4.10
- net at U4.E3 (IO_L11P_T1_SRCC_35): now also J4.12
- net at U4.E5 (IO_L13N_T2_MRCC_35): now also J4.17
- net at U4.F2 (IO_L15P_T2_DQS_35): now also J4.20
- net at U4.F3 (IO_L14N_T2_SRCC_35): now also J4.19
- net at U4.F4 (IO_L14P_T2_SRCC_35): now also J4.18
- net at U4.F5 (IO_L13P_T2_MRCC_35): now also J4.16
- net at U4.G1 (IO_L17N_T2_35): now also J4.25
- net at U4.G2 (IO_L17P_T2_35): now also J4.24
- net at U4.G4 (IO_L16N_T2_35): now also J4.23
- net at U4.G5 (IO_L16P_T2_35): now also J4.22
- net at U4.H1 (IO_L20N_T3_35): now also J4.31
- net at U4.H2 (IO_L20P_T3_35): now also J4.30
- net at U4.H3 (IO_L21N_T3_DQS_35): now also J4.33
- net at U4.H4 (IO_L18N_T2_35): now also J4.27
- net at U4.H5 (IO_L18P_T2_35): now also J4.26
- net at U4.J1 (IO_L22N_T3_35): now also J4.35
- net at U4.J3 (IO_L21P_T3_DQS_35): now also J4.32
- net at U4.J4 (IO_L19N_T3_VREF_35): now also J4.29
- net at U4.J5 (IO_L19P_T3_35): now also J4.28
- net at U4.K1 (IO_L22P_T3_35): now also J4.34
- net at U4.K2 (IO_L24N_T3_35): now also J4.39
- net at U4.K3 (IO_L24P_T3_35): now also J4.38
- net at U4.K5 (IO_25_35): now also J4.40
- net at U4.L2 (IO_L23N_T3_35): now also J4.37
- net at U4.L3 (IO_L23P_T3_35): now also J4.36
Other:
- moved on the sheet: C24, C25, C26, C27, C28, C29, C30, C31, C32, C33, C34, C35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

Commit message: Some error fix
Connections:
- net +3V3 is gone; now on net +3.3V: J1.2, R16.1, R17.2, R18.2, R19.2, R20.1, U4.E7 (CFGBVS_0), U4.M9 (M0_0)
Other:
- moved on the sheet: R19
