File: PCB/fpga.kicad_sch (KiCad schematic)
At the start: 22 parts, among them IC1 S25FL256LAGMFI003, IC2 LT1932ES6#TRMPBF, J1 0878311420, J4 62684-402100ALF, U4 XC7A100T-FTG256, U5 IS62C1024AL-35QLI-TR, Y2 ECS-3953M-400-BN-TR

Commit message: Pcb
Parts:
- U4: footprint fpga:BGA256C100P16X16_1700X1700X155 -> fpga_real:BGA256C100P16X16_1700X1700X155
Connections:
- net at J4.35: no longer U4.J1 (IO_L22N_T3_35)
- net at J4.36: no longer U4.L3 (IO_L23P_T3_35)
- net at J4.37: no longer U4.L2 (IO_L23N_T3_35)
- net at J4.38: no longer U4.K3 (IO_L24P_T3_35)
- net at J4.39: no longer U4.K2 (IO_L24N_T3_35)
- net at J4.40: no longer U4.K5 (IO_25_35)
- no-connect marks 81 -> 93
Changed lines of the file:
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@@
   (no_connect (at 374.65 137.16))
   (no_connect (at 273.05 165.1))
+  (no_connect (at 381 236.22))
   (no_connect (at 93.98 82.55))
   (no_connect (at 93.98 148.59))
   (no_connect (at 374.65 134.62))
   (no_connect (at 93.98 115.57))
+  (no_connect (at 381 246.38))
   (no_connect (at 93.98 118.11))
   (no_connect (at 93.98 72.39))
@@
   (no_connect (at 167.64 92.71))
   (no_connect (at 93.98 133.35))
+  (no_connect (at 374.65 236.22))
+  (no_connect (at 381 243.84))
   (no_connect (at 93.98 67.31))
   (no_connect (at 93.98 125.73))
@@
   (no_connect (at 273.05 170.18))
   (no_connect (at 74.93 50.8))
+  (no_connect (at 374.65 233.68))
   (no_connect (at 374.65 154.94))
   (no_connect (at 93.98 161.29))
@@
   (no_connect (at 374.65 142.24))
   (no_connect (at 167.64 85.09))
+  (no_connect (at 381 233.68))
+  (no_connect (at 374.65 246.38))
   (no_connect (at 93.98 95.25))
   (no_connect (at 93.98 41.91))
@@
   (no_connect (at 93.98 166.37))
   (no_connect (at 273.05 167.64))
+  (no_connect (at 374.65 243.84))
   (no_connect (at 93.98 107.95))
   (no_connect (at 93.98 100.33))
+  (no_connect (at 381 238.76))
   (no_connect (at 93.98 90.17))
   (no_connect (at 93.98 85.09))
   (no_connect (at 93.98 113.03))
+  (no_connect (at 374.65 241.3))
   (no_connect (at 93.98 135.89))
   (no_connect (at 93.98 87.63))
   (no_connect (at 93.98 140.97))
   (no_connect (at 167.64 77.47))
+  (no_connect (at 381 241.3))
   (no_connect (at 167.64 90.17))
   (no_connect (at 93.98 151.13))
   (no_connect (at 74.93 48.26))
+  (no_connect (at 374.65 238.76))
   (no_connect (at 93.98 163.83))
   (no_connect (at 93.98 59.69))
@@
     (stroke (width 0) (type default))
   )
-  (wire (pts (xy 374.65 243.84) (xy 381 243.84))
-    (stroke (width 0) (type default))
-  )
   (wire (pts (xy 374.65 215.9) (xy 381 215.9))
     (stroke (width 0) (type default))
@@
     (stroke (width 0) (type default))
   )
-  (wire (pts (xy 374.65 233.68) (xy 381 233.68))
-    (stroke (width 0) (type default))
-  )
-  (wire (pts (xy 374.65 241.3) (xy 381 241.3))
-    (stroke (width 0) (type default))
-  )
   (wire (pts (xy 224.79 118.11) (xy 167.64 118.11))
     (stroke (width 0) (type default))
@@
     (stroke (width 0) (type default))
   )
-  (wire (pts (xy 374.65 238.76) (xy 381 238.76))
-    (stroke (width 0) (type default))
-  )
   (wire (pts (xy 90.17 27.94) (xy 90.17 44.45))
     (stroke (width 0) (type default))
@@
     (stroke (width 0) (type default))
   )
-  (wire (pts (xy 374.65 246.38) (xy 381 246.38))
-    (stroke (width 0) (type default))
-  )
   (wire (pts (xy 43.18 114.3) (xy 45.72 114.3))
     (stroke (width 0) (type default))
@@
     (stroke (width 0) (type default))
   )
-  (wire (pts (xy 374.65 236.22) (xy 381 236.22))
-    (stroke (width 0) (type default))
-  )
   (wire (pts (xy 168.91 130.81) (xy 168.91 129.54))
     (stroke (width 0) (type default))
@@
       (effects (font (size 1.27 1.27)))
     )
-    (property "Footprint" "fpga:BGA256C100P16X16_1700X1700X155" (at 138.43 95.25 0)
+    (property "Footprint" "fpga_real:BGA256C100P16X16_1700X1700X155" (at 138.43 95.25 0)
       (effects (font (size 1.27 1.27)) hide)
     )
@@
       (effects (font (size 1.27 1.27)))
     )
-    (property "Footprint" "fpga:BGA256C100P16X16_1700X1700X155" (at 262.89 54.61 0)
+    (property "Footprint" "fpga_real:BGA256C100P16X16_1700X1700X155" (at 262.89 54.61 0)
       (effects (font (size 1.27 1.27)) hide)
     )
@@
       (effects (font (size 1.27 1.27)))
     )
-    (property "Footprint" "fpga:BGA256C100P16X16_1700X1700X155" (at 323.85 175.26 0)
+    (property "Footprint" "fpga_real:BGA256C100P16X16_1700X1700X155" (at 323.85 175.26 0)
       (effects (font (size 1.27 1.27)) hide)
     )
@@
       (effects (font (size 1.27 1.27)))
     )
-    (property "Footprint" "fpga:BGA256C100P16X16_1700X1700X155" (at 74.93 111.76 0)
+    (property "Footprint" "fpga_real:BGA256C100P16X16_1700X1700X155" (at 74.93 111.76 0)
       (effects (font (size 1.27 1.27)) hide)
     )
