File: PCB/power_supply.kicad_sch (KiCad schematic)
At the start: 32 parts, among them U1 TPS54325, U2 TPS54294

Commit message: Adding unit C and D to FPGA (Stil missing unit B)
Parts:
- U1: footprint (none) -> Package_SO:TSSOP-14-1EP_4.4x5mm_P0.65mm
- U2: footprint (none) -> Package_SO:HTSSOP-16-1EP_4.4x5mm_P0.65mm_EP3x3mm
Connections:
- no-connect marks 0 -> 1
Changed lines of the file:
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@@
   (junction (at 157.48 81.28) (diameter 0) (color 0 0 0 0)
   )
+  (no_connect (at 144.78 116.84))
   (wire (pts (xy 153.67 121.92) (xy 153.67 125.73))
     (stroke (width 0) (type default))
@@
       (effects (font (size 1.27 1.27)))
     )
-    (property "Footprint" "" (at 133.35 111.76 0)
+    (property "Footprint" "Package_SO:HTSSOP-16-1EP_4.4x5mm_P0.65mm_EP3x3mm" (at 133.35 111.76 0)
       (effects (font (size 1.27 1.27)) hide)
     )
@@
       (effects (font (size 1.27 1.27)))
     )
-    (property "Footprint" "" (at 133.35 59.69 0)
-      (effects (font (size 1.27 1.27)) hide)
-    )
+    (property "Footprint" "Package_SO:TSSOP-14-1EP_4.4x5mm_P0.65mm" (at 133.35 59.69 0)
+      (effects (font (size 1.27 1.27)) hide)
+    )

Commit message: Work
Parts:
- added J2: USB_B_Micro, symbol Connector:USB_B_Micro
Connections:
- net GND: now also J2.5 (GND)
- net 5V_OUT: now reaches C10.1, C11.1, C12.1, C13.1, C2.1, C3.1, C4.1, U1.13 (VIN), U1.14 (VCC), U2.1 (VIN1), U2.16 (VIN2)
- net 5V_OUT: now also J2.1 (VBUS)
Changed lines of the file:
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@@
   (junction (at 226.06 113.03) (diameter 0) (color 0 0 0 0)
   )
+  (junction (at 74.93 53.34) (diameter 0) (color 0 0 0 0)
+  )
   (junction (at 157.48 113.03) (diameter 0) (color 0 0 0 0)
   )
@@
   )
   (junction (at 77.47 109.22) (diameter 0) (color 0 0 0 0)
+  )
+  (junction (at 81.28 53.34) (diameter 0) (color 0 0 0 0)
   )
   (junction (at 171.45 138.43) (diameter 0) (color 0 0 0 0)
@@
     (stroke (width 0) (type default))
   )
+  (wire (pts (xy 74.93 46.99) (xy 74.93 53.34))
+    (stroke (width 0) (type default))
+  )
   (wire (pts (xy 114.3 68.58) (xy 114.3 60.96))
     (stroke (width 0) (type default))
@@
     (stroke (width 0) (type default))
   )
+  (wire (pts (xy 74.93 53.34) (xy 81.28 53.34))
+    (stroke (width 0) (type default))
+  )
   (wire (pts (xy 180.34 138.43) (xy 204.47 138.43))
     (stroke (width 0) (type default))
@@
     (stroke (width 0) (type default))
   )
+  (wire (pts (xy 71.12 53.34) (xy 74.93 53.34))
+    (stroke (width 0) (type default))
+  )
   (wire (pts (xy 86.36 81.28) (xy 92.71 81.28))
     (stroke (width 0) (type default))
@@
   (wire (pts (xy 93.98 106.68) (xy 93.98 138.43))
     (stroke (width 0) (type default))
+  )
+  (hierarchical_label "5V_OUT" (shape input) (at 74.93 46.99 0) (fields_autoplaced)
+    (effects (font (size 1.27 1.27)) (justify left))
   )
   (symbol (lib_id "Device:R") (at 161.29 129.54 0) (unit 1)
@@
     )
   )
+  (symbol (lib_id "power:GND") (at 63.5 68.58 0) (unit 1)
+    (in_bom yes) (on_board yes) (dnp no) (fields_autoplaced)
+    (property "Reference" "#PWR049" (at 63.5 74.93 0)
+      (effects (font (size 1.27 1.27)) hide)
+    )
+    (property "Value" "GND" (at 63.5 73.66 0)
+      (effects (font (size 1.27 1.27)))
+    )
+    (property "Footprint" "" (at 63.5 68.58 0)
+      (effects (font (size 1.27 1.27)) hide)
+    )
+    (property "Datasheet" "" (at 63.5 68.58 0)
+      (effects (font (size 1.27 1.27)) hide)
+    )
+    (pin "1")
+    (instances
+      (project "PCB"
+        (path "/aa113cd6-c3ac-4890-9a84-1ea195994408/854a1da6-0a91-483b-964f-5f1aec25ba6d"
+          (reference "#PWR049") (unit 1)
+        )
+      )
+    )
+  )
   (symbol (lib_id "power:+1V0") (at 207.01 49.53 0) (unit 1)
     (in_bom yes) (on_board yes) (dnp no) (fields_autoplaced)
@@
         )
       )
+    )
+  )
+  (symbol (lib_id "Connector:USB_B_Micro") (at 63.5 58.42 0) (unit 1)
+    (in_bom yes) (on_board yes) (dnp no) (fields_autoplaced)
+    (property "Reference" "J2" (at 63.5 45.72 0)
+      (effects (font (size 1.27 1.27)))
+    )
+    (property "Value" "USB_B_Micro" (at 63.5 48.26 0)
+      (effects (font (size 1.27 1.27)))
+    )
+    (property "Footprint" "" (at 67.31 59.69 0)
+      (effects (font (size 1.27 1.27)) hide)
+    )
+    (property "Datasheet" "~" (at 67.31 59.69 0)
+      (effects (font (size 1.27 1.27)) hide)
+    )
+    (pin "1")
+    (pin "2")
+    (pin "3")
+    (pin "4")
+    (pin "5")
+    (pin "6")
+    (instances
+      (project "PCB"
+        (path "/aa113cd6-c3ac-4890-9a84-1ea195994408/854a1da6-0a91-483b-964f-5f1aec25ba6d"
+          (reference "J2") (unit 1)
+        )
+      )

Commit message: work
Connections:
- net 5V_OUT: now also U1.7 (EN)
- no-connect marks 1 -> 5
Changed lines of the file:
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@@
   (junction (at 71.12 109.22) (diameter 0) (color 0 0 0 0)
   )
+  (junction (at 121.92 55.88) (diameter 0) (color 0 0 0 0)
+  )
   (junction (at 107.95 58.42) (diameter 0) (color 0 0 0 0)
   )
@@
   (junction (at 157.48 81.28) (diameter 0) (color 0 0 0 0)
   )
+  (no_connect (at 71.12 58.42))
+  (no_connect (at 60.96 68.58))
   (no_connect (at 144.78 116.84))
+  (no_connect (at 71.12 63.5))
+  (no_connect (at 71.12 60.96))
   (wire (pts (xy 153.67 121.92) (xy 153.67 125.73))
     (stroke (width 0) (type default))
@@
     (stroke (width 0) (type default))
   )
+  (wire (pts (xy 120.65 66.04) (xy 120.65 55.88))
+    (stroke (width 0) (type default))
+  )
   (wire (pts (xy 149.86 106.68) (xy 149.86 101.6))
     (stroke (width 0) (type default))
@@
     (stroke (width 0) (type default))
   )
+  (wire (pts (xy 120.65 55.88) (xy 121.92 55.88))
+    (stroke (width 0) (type default))
+  )
   (wire (pts (xy 144.78 53.34) (xy 147.32 53.34))
     (stroke (width 0) (type default))
@@
     (stroke (width 0) (type default))
   )
+  (wire (pts (xy 121.92 66.04) (xy 120.65 66.04))
+    (stroke (width 0) (type default))
+  )

Commit message: pls work
Changed lines of the file:
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@@
       (effects (font (size 1.27 1.27)) (justify left))
     )
-    (property "Value" "22.1k" (at 64.77 130.81 0)
+    (property "Value" "22.1k" (at 57.785 132.715 0)
       (effects (font (size 1.27 1.27)) (justify left))
     )
@@
       (effects (font (size 1.27 1.27)) (justify left))
     )
-    (property "Value" "30.1k" (at 63.5 118.11 0)
-      (effects (font (size 1.27 1.27)) (justify left))
-    )
+    (property "Value" "30.1k" (at 58.42 118.11 0)
+      (effects (font (size 1.27 1.27)) (justify left))
+    )

Commit message: Footprints
Parts:
- C1, C10, C11, C12, C13, C14, C15, C16, C17, C18, C19, C2, C3, C4, C5, C6, C7, C8, C9: footprint (none) -> Capacitor_SMD:C_0805_2012Metric_Pad1.18x1.45mm_HandSolder
- J2: footprint (none) -> 10118193-0001LF:AMPHENOL_10118193-0001LF
- R1, R2, R3, R4, R5, R6, R7, R8: footprint (none) -> Resistor_SMD:R_0805_2012Metric_Pad1.20x1.40mm_HandSolder
Changed lines of the file:
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@@
       (effects (font (size 1.27 1.27)) (justify left))
     )
-    (property "Footprint" "" (at 159.512 129.54 90)
+    (property "Footprint" "Resistor_SMD:R_0805_2012Metric_Pad1.20x1.40mm_HandSolder" (at 159.512 129.54 90)
       (effects (font (size 1.27 1.27)) hide)
     )
@@
       (effects (font (size 1.27 1.27)) (justify left))
     )
-    (property "Footprint" "" (at 106.172 73.66 90)
+    (property "Footprint" "Resistor_SMD:R_0805_2012Metric_Pad1.20x1.40mm_HandSolder" (at 106.172 73.66 90)
       (effects (font (size 1.27 1.27)) hide)
     )
@@
       (effects (font (size 1.27 1.27)) (justify left))
     )
-    (property "Footprint" "" (at 94.9452 106.68 0)
+    (property "Footprint" "Capacitor_SMD:C_0805_2012Metric_Pad1.18x1.45mm_HandSolder" (at 94.9452 106.68 0)
       (effects (font (size 1.27 1.27)) hide)
     )
@@
       (effects (font (size 1.27 1.27)) (justify left))
     )
-    (property "Footprint" "" (at 158.4452 111.76 0)
+    (property "Footprint" "Capacitor_SMD:C_0805_2012Metric_Pad1.18x1.45mm_HandSolder" (at 158.4452 111.76 0)
       (effects (font (size 1.27 1.27)) hide)
     )
@@
       (effects (font (size 1.27 1.27)) (justify left))
     )
-    (property "Footprint" "" (at 154.6352 133.35 0)
+    (property "Footprint" "Capacitor_SMD:C_0805_2012Metric_Pad1.18x1.45mm_HandSolder" (at 154.6352 133.35 0)
       (effects (font (size 1.27 1.27)) hide)
     )
@@
       (effects (font (size 1.27 1.27)) (justify left))
     )
-    (property "Footprint" "" (at 116.5352 76.2 0)
+    (property "Footprint" "Capacitor_SMD:C_0805_2012Metric_Pad1.18x1.45mm_HandSolder" (at 116.5352 76.2 0)
       (effects (font (size 1.27 1.27)) hide)
     )
@@
       (effects (font (size 1.27 1.27)) (justify left))
     )
-    (property "Footprint" "" (at 158.4452 76.2 0)
+    (property "Footprint" "Capacitor_SMD:C_0805_2012Metric_Pad1.18x1.45mm_HandSolder" (at 158.4452 76.2 0)
       (effects (font (size 1.27 1.27)) hide)
     )
@@
       (effects (font (size 1.27 1.27)) (justify left))
     )
-    (property "Footprint" "" (at 195.2752 60.96 0)
+    (property "Footprint" "Capacitor_SMD:C_0805_2012Metric_Pad1.18x1.45mm_HandSolder" (at 195.2752 60.96 0)
       (effects (font (size 1.27 1.27)) hide)
     )
@@
       (effects (font (size 1.27 1.27)) (justify left))
     )
-    (property "Footprint" "" (at 102.5652 106.68 0)
+    (property "Footprint" "Capacitor_SMD:C_0805_2012Metric_Pad1.18x1.45mm_HandSolder" (at 102.5652 106.68 0)
       (effects (font (size 1.27 1.27)) hide)
     )
@@
       (effects (font (size 1.27 1.27)) (justify left))
     )
-    (property "Footprint" "" (at 224.282 128.27 90)
+    (property "Footprint" "Resistor_SMD:R_0805_2012Metric_Pad1.20x1.40mm_HandSolder" (at 224.282 128.27 90)
       (effects (font (size 1.27 1.27)) hide)
     )
@@
       (effects (font (size 1.27 1.27)) (justify left))
     )
-    (property "Footprint" "" (at 181.3052 107.95 0)
+    (property "Footprint" "Capacitor_SMD:C_0805_2012Metric_Pad1.18x1.45mm_HandSolder" (at 181.3052 107.95 0)
       (effects (font (size 1.27 1.27)) hide)
     )
@@
       (effects (font (size 1.27 1.27)) (justify left))
     )
-    (property "Footprint" "" (at 62.992 130.81 90)
+    (property "Footprint" "Resistor_SMD:R_0805_2012Metric_Pad1.20x1.40mm_HandSolder" (at 62.992 130.81 90)
       (effects (font (size 1.27 1.27)) hide)
     )
@@
       (effects (font (size 1.27 1.27)) (justify left))
     )
-    (property "Footprint" "" (at 111.4552 110.49 0)
+    (property "Footprint" "Capacitor_SMD:C_0805_2012Metric_Pad1.18x1.45mm_HandSolder" (at 111.4552 110.49 0)
       (effects (font (size 1.27 1.27)) hide)
     )
@@
       (effects (font (size 1.27 1.27)) (justify left))
     )
-    (property "Footprint" "" (at 87.3252 60.96 0)
+    (property "Footprint" "Capacitor_SMD:C_0805_2012Metric_Pad1.18x1.45mm_HandSolder" (at 87.3252 60.96 0)
       (effects (font (size 1.27 1.27)) hide)
     )
@@
       (effects (font (size 1.27 1.27)) (justify left))
     )
-    (property "Footprint" "" (at 224.282 118.11 90)
+    (property "Footprint" "Resistor_SMD:R_0805_2012Metric_Pad1.20x1.40mm_HandSolder" (at 224.282 118.11 90)
       (effects (font (size 1.27 1.27)) hide)
     )
@@
       (effects (font (size 1.27 1.27)))
     )
-    (property "Footprint" "" (at 163.83 65.278 90)
+    (property "Footprint" "Resistor_SMD:R_0805_2012Metric_Pad1.20x1.40mm_HandSolder" (at 163.83 65.278 90)
       (effects (font (size 1.27 1.27)) hide)
     )
@@
       (effects (font (size 1.27 1.27)) (justify left))
     )
-    (property "Footprint" "" (at 214.3252 120.65 0)
+    (property "Footprint" "Capacitor_SMD:C_0805_2012Metric_Pad1.18x1.45mm_HandSolder" (at 214.3252 120.65 0)
       (effects (font (size 1.27 1.27)) hide)
     )
@@
       (effects (font (size 1.27 1.27)))
     )
-    (property "Footprint" "" (at 67.31 59.69 0)
+    (property "Footprint" "10118193-0001LF:AMPHENOL_10118193-0001LF" (at 67.31 59.69 0)
       (effects (font (size 1.27 1.27)) hide)
     )
@@
       (effects (font (size 1.27 1.27)))
     )
-    (property "Footprint" "" (at 181.61 57.4548 0)
+    (property "Footprint" "Capacitor_SMD:C_0805_2012Metric_Pad1.18x1.45mm_HandSolder" (at 181.61 57.4548 0)
       (effects (font (size 1.27 1.27)) hide)
     )
@@
       (effects (font (size 1.27 1.27)) (justify left))
     )
-    (property "Footprint" "" (at 172.4152 107.95 0)
+    (property "Footprint" "Capacitor_SMD:C_0805_2012Metric_Pad1.18x1.45mm_HandSolder" (at 172.4152 107.95 0)
       (effects (font (size 1.27 1.27)) hide)
     )
@@
       (effects (font (size 1.27 1.27)) (justify left))
     )
-    (property "Footprint" "" (at 72.0852 124.46 0)
+    (property "Footprint" "Capacitor_SMD:C_0805_2012Metric_Pad1.18x1.45mm_HandSolder" (at 72.0852 124.46 0)
       (effects (font (size 1.27 1.27)) hide)
     )
@@
       (effects (font (size 1.27 1.27)) (justify left))
     )
-    (property "Footprint" "" (at 205.4352 120.65 0)
+    (property "Footprint" "Capacitor_SMD:C_0805_2012Metric_Pad1.18x1.45mm_HandSolder" (at 205.4352 120.65 0)
       (effects (font (size 1.27 1.27)) hide)
     )
@@
       (effects (font (size 1.27 1.27)) (justify left))
     )
-    (property "Footprint" "" (at 100.0252 60.96 0)
+    (property "Footprint" "Capacitor_SMD:C_0805_2012Metric_Pad1.18x1.45mm_HandSolder" (at 100.0252 60.96 0)
       (effects (font (size 1.27 1.27)) hide)
     )
@@
       (effects (font (size 1.27 1.27)) (justify left))
     )
-    (property "Footprint" "" (at 93.6752 60.96 0)
+    (property "Footprint" "Capacitor_SMD:C_0805_2012Metric_Pad1.18x1.45mm_HandSolder" (at 93.6752 60.96 0)
       (effects (font (size 1.27 1.27)) hide)
     )
@@
       (effects (font (size 1.27 1.27)) (justify left))
     )
-    (property "Footprint" "" (at 106.172 63.5 90)
+    (property "Footprint" "Resistor_SMD:R_0805_2012Metric_Pad1.20x1.40mm_HandSolder" (at 106.172 63.5 90)
       (effects (font (size 1.27 1.27)) hide)
     )
@@
       (effects (font (size 1.27 1.27)) (justify left))
     )
-    (property "Footprint" "" (at 78.4352 124.46 0)
+    (property "Footprint" "Capacitor_SMD:C_0805_2012Metric_Pad1.18x1.45mm_HandSolder" (at 78.4352 124.46 0)
       (effects (font (size 1.27 1.27)) hide)
     )
@@
       (effects (font (size 1.27 1.27)) (justify left))
     )
-    (property "Footprint" "" (at 62.992 116.84 90)
+    (property "Footprint" "Resistor_SMD:R_0805_2012Metric_Pad1.20x1.40mm_HandSolder" (at 62.992 116.84 90)
       (effects (font (size 1.27 1.27)) hide)
     )
@@
       (effects (font (size 1.27 1.27)) (justify left))
     )
-    (property "Footprint" "" (at 202.8952 60.96 0)
-      (effects (font (size 1.27 1.27)) hide)
-    )
+    (property "Footprint" "Capacitor_SMD:C_0805_2012Metric_Pad1.18x1.45mm_HandSolder" (at 202.8952 60.96 0)
+      (effects (font (size 1.27 1.27)) hide)
+    )

Commit message: Start PCB
Parts:
- L1, L2, L3: footprint (none) -> Inductor_SMD:L_0805_2012Metric_Pad1.15x1.40mm_HandSolder
Changed lines of the file:
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@@
       (effects (font (size 1.27 1.27)))
     )
-    (property "Footprint" "" (at 187.96 53.34 0)
+    (property "Footprint" "Inductor_SMD:L_0805_2012Metric_Pad1.15x1.40mm_HandSolder" (at 187.96 53.34 0)
       (effects (font (size 1.27 1.27)) hide)
     )
@@
       (effects (font (size 1.27 1.27)))
     )
-    (property "Footprint" "" (at 83.82 109.22 0)
+    (property "Footprint" "Inductor_SMD:L_0805_2012Metric_Pad1.15x1.40mm_HandSolder" (at 83.82 109.22 0)
       (effects (font (size 1.27 1.27)) hide)
     )
@@
       (effects (font (size 1.27 1.27)))
     )
-    (property "Footprint" "" (at 191.77 113.03 0)
-      (effects (font (size 1.27 1.27)) hide)
-    )
+    (property "Footprint" "Inductor_SMD:L_0805_2012Metric_Pad1.15x1.40mm_HandSolder" (at 191.77 113.03 0)
+      (effects (font (size 1.27 1.27)) hide)
+    )

Commit message: more
Parts:
- added JP1, JP2: Jumper_2_Bridged, TestPoint:TestPoint_2Pads_Pitch2.54mm_Drill0.8mm, symbol Jumper:Jumper_2_Bridged
- added JP3: Jumper_2_Bridged, symbol Jumper:Jumper_2_Bridged
Connections:
- net +1V0: now also JP1.2 (B); no longer C6.1, C7.1, L1.2, R2.1, U1.1 (VO)
- net +1V8: now also JP3.2 (B); no longer C15.1, C16.1, L2.1, R5.1
- net +3.3V: now also JP2.2 (B); no longer C17.1, C18.1, L3.2, R7.1
- new net: C6.1, C7.1, JP1.1 (A), L1.2, R2.1, U1.1 (VO)
- new net: C15.1, C16.1, JP3.1 (A), L2.1, R5.1
- new net: C17.1, C18.1, JP2.1 (A), L3.2, R7.1
