File: PCB/power_supply.kicad_sch (KiCad schematic)
At the start: 36 parts, among them J2 USB_B_Micro, U1 TPS54325, U2 TPS54294

Commit message: PCB
Parts:
- JP3: footprint (none) -> TestPoint:TestPoint_2Pads_Pitch2.54mm_Drill0.8mm
Connections:
- net GND: now also C1.2, C19.2, C2.2, C3.2, C4.2, C6.2, C7.2, R3.2, U1.5 (GND), U1.8 (PGND1), U1.9 (PGND2)
Changed lines of the file:
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@@
   (junction (at 121.92 55.88) (diameter 0) (color 0 0 0 0)
+  )
+  (junction (at 133.35 81.28) (diameter 0) (color 0 0 0 0)
   )
   (junction (at 107.95 58.42) (diameter 0) (color 0 0 0 0)
@@
     (stroke (width 0) (type default))
   )
-  (wire (pts (xy 121.92 81.28) (xy 144.78 81.28))
+  (wire (pts (xy 121.92 81.28) (xy 133.35 81.28))
     (stroke (width 0) (type default))
   )
@@
     (stroke (width 0) (type default))
   )
+  (wire (pts (xy 133.35 82.55) (xy 133.35 81.28))
+    (stroke (width 0) (type default))
+  )
   (wire (pts (xy 147.32 104.14) (xy 144.78 104.14))
     (stroke (width 0) (type default))
@@
     (stroke (width 0) (type default))
   )
+  (wire (pts (xy 133.35 81.28) (xy 144.78 81.28))
+    (stroke (width 0) (type default))
+  )
   (wire (pts (xy 194.31 53.34) (xy 191.77 53.34))
     (stroke (width 0) (type default))
@@
     (stroke (width 0) (type default))
   )
-  (wire (pts (xy 236.22 113.03) (xy 237.49 113.03))
+  (wire (pts (xy 236.22 113.03) (xy 248.92 113.03))
     (stroke (width 0) (type default))
   )
@@
     (stroke (width 0) (type default))
   )
-  (wire (pts (xy 133.35 72.39) (xy 133.35 82.55))
+  (wire (pts (xy 133.35 72.39) (xy 133.35 81.28))
     (stroke (width 0) (type default))
   )
@@
     )
   )
-  (symbol (lib_id "power:+3.3V") (at 237.49 113.03 0) (unit 1)
-    (in_bom yes) (on_board yes) (dnp no) (fields_autoplaced)
-    (property "Reference" "#PWR05" (at 237.49 116.84 0)
-      (effects (font (size 1.27 1.27)) hide)
-    )
-    (property "Value" "+3.3V" (at 237.49 107.95 0)
-      (effects (font (size 1.27 1.27)))
-    )
-    (property "Footprint" "" (at 237.49 113.03 0)
-      (effects (font (size 1.27 1.27)) hide)
-    )
-    (property "Datasheet" "" (at 237.49 113.03 0)
+  (symbol (lib_id "power:+3.3V") (at 248.92 113.03 0) (unit 1)
+    (in_bom yes) (on_board yes) (dnp no) (fields_autoplaced)
+    (property "Reference" "#PWR05" (at 248.92 116.84 0)
+      (effects (font (size 1.27 1.27)) hide)
+    )
+    (property "Value" "+3.3V" (at 248.92 107.95 0)
+      (effects (font (size 1.27 1.27)))
+    )
+    (property "Footprint" "" (at 248.92 113.03 0)
+      (effects (font (size 1.27 1.27)) hide)
+    )
+    (property "Datasheet" "" (at 248.92 113.03 0)
       (effects (font (size 1.27 1.27)) hide)
     )
@@
       (effects (font (size 1.27 1.27)))
     )
-    (property "Footprint" "" (at 59.69 109.22 0)
-      (effects (font (size 1.27 1.27)) hide)
-    )
+    (property "Footprint" "TestPoint:TestPoint_2Pads_Pitch2.54mm_Drill0.8mm" (at 59.69 109.22 0)
+      (effects (font (size 1.27 1.27)) hide)
+    )
