File: PCB/PCB.kicad_pcb (KiCad board)
At the start: 2 copper layers, 151 parts, among them IC1 S25FL256LAGMFI003, J1 0878311420, J2 USB_B_Micro, J4 62684-402100ALF, J5 L77HDE15SD1CH4FVGA, J6 USB1130-15-A_REVA, SW1 SW_Push, SW2 SW_Push, SW3 SW_Push, SW4 SW_Push, U1 TPS54325, U2 TPS54294, U3 COM-09032, U4 XC7A100T-FTG256, U5 IS62C1024AL-35QLI-TR, Y1 Crystal_GND24, Y2 ECS-3953M-400-BN-TR

Commit message: more
Parts:
- moved U5 184.3 mm to (286.6, -58.0)
- moved J4 181.3 mm to (263.7, -80.9)
- moved C23 181.3 mm to (242.4, -71.2)
- moved R14 181.3 mm to (313.5, -140.1)
- moved C1 181.3 mm to (364.1, -58.3)
- moved C15 181.3 mm to (365.3, -98.7)
- moved C16 181.3 mm to (365.3, -95.6)
- moved C17 181.3 mm to (365.3, -92.6)
- moved C18 181.3 mm to (365.3, -89.6)
- moved C19 181.3 mm to (365.3, -86.6)
- moved C2 181.3 mm to (364.1, -55.3)
- moved C20 181.3 mm to (215.5, -111.8)
- moved C21 181.3 mm to (215.5, -108.8)
- moved C22 181.3 mm to (215.5, -105.8)
- moved C24 181.3 mm to (379.1, -116.2)
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Other:
- board outline added: 255 x 147 mm
- copper layers 2 -> 6

Commit message: PCB
Parts:
- added C93: 1u, Capacitor_SMD:C_0805_2012Metric_Pad1.18x1.45mm_HandSolder, F.Cu at (30.4, 146.4)
- added C94: 100u, Capacitor_SMD:C_0805_2012Metric_Pad1.18x1.45mm_HandSolder, F.Cu at (42.8, 151.0)
- added C95: 4.7u, Capacitor_SMD:C_0805_2012Metric_Pad1.18x1.45mm_HandSolder, F.Cu at (238.5, 38.0)
- added C96: 1u, Capacitor_SMD:C_0805_2012Metric_Pad1.18x1.45mm_HandSolder, F.Cu at (239.7, 44.2)
- added D2: MBR0520, Diode_SMD:D_SOD-123, F.Cu at (231.3, 32.2)
- added IC2: LT1932ES6#TRMPBF, ledDriver:SOT95P280X100-6N, F.Cu at (226.4, 37.0)
- added JP1: Jumper_2_Bridged, TestPoint:TestPoint_2Pads_Pitch2.54mm_Drill0.8mm, F.Cu at (93.8, 136.0)
- added JP2: Jumper_2_Bridged, TestPoint:TestPoint_2Pads_Pitch2.54mm_Drill0.8mm, F.Cu at (126.2, 127.8)
- added JP3: Jumper_2_Bridged, TestPoint:TestPoint_2Pads_Pitch2.54mm_Drill0.8mm, F.Cu at (91.2, 115.0)
- added L4: 6.8u, Inductor_SMD:L_0805_2012Metric_Pad1.05x1.20mm_HandSolder, F.Cu at (230.8, 40.0)
- added R38: 15, Resistor_SMD:R_0805_2012Metric_Pad1.20x1.40mm_HandSolder, F.Cu at (243.2, 32.0)
- added R39: 15, Resistor_SMD:R_0805_2012Metric_Pad1.20x1.40mm_HandSolder, F.Cu at (243.2, 35.0)
- added R40: 562, Resistor_SMD:R_0805_2012Metric_Pad1.20x1.40mm_HandSolder, F.Cu at (236.5, 32.0)
- moved C24 468.3 mm to (-42.1, 88.5)
- moved C25 468.3 mm to (-42.1, 91.5)
- moved C26 468.3 mm to (-42.1, 94.5)
- moved C27 468.3 mm to (-42.1, 97.5)
- moved C28 468.3 mm to (-42.1, 100.6)
- moved C29 468.3 mm to (-42.1, 103.6)
- moved C30 468.3 mm to (-42.1, 106.6)
- moved C31 468.3 mm to (-42.1, 109.6)
- moved C32 468.3 mm to (-42.1, 112.6)
- moved C33 468.3 mm to (-42.1, 115.6)
- moved C34 468.3 mm to (-42.1, 118.6)
- moved C35 419.7 mm to (-16.8, 91.7)
- moved C36 419.7 mm to (-16.8, 94.7)
- moved C37 419.7 mm to (-16.8, 97.7)
- moved C38 419.7 mm to (-16.8, 100.7)
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Connections:
- C1 pad 1: +1V8 -> Net-(JP3-A)
- C11 pad 2: Net-(U1-GND) -> GND
- C16 pad 1: +1V0 -> Net-(JP1-A)
- C16 pad 2: Net-(U1-GND) -> GND
- C17 pad 1: +1V0 -> Net-(JP1-A)
- C17 pad 2: Net-(U1-GND) -> GND
- C18 pad 1: +3.3V -> Net-(JP2-A)
- C19 pad 1: +3.3V -> Net-(JP2-A)
- C2 pad 1: +1V8 -> Net-(JP3-A)
- C3 pad 2: Net-(U1-GND) -> GND
- C4 pad 2: Net-(U1-GND) -> GND
- C6 pad 2: Net-(U1-GND) -> GND
- C9 pad 2: Net-(U1-GND) -> GND
- DEBUG_HEADER1 pad 12: Net-(DEBUG_HEADER1-TRACECLK) -> unconnected-(DEBUG_HEADER1-TRACECLK-Pad12)
- DEBUG_HEADER1 pad 14: Net-(DEBUG_HEADER1-TRACEDATA[0]) -> unconnected-(DEBUG_HEADER1-TRACEDATA[0]-Pad14)
- DEBUG_HEADER1 pad 16: Net-(DEBUG_HEADER1-TRACEDATA[1]) -> unconnected-(DEBUG_HEADER1-TRACEDATA[1]-Pad16)
- DEBUG_HEADER1 pad 18: Net-(DEBUG_HEADER1-TRACEDATA[2]) -> unconnected-(DEBUG_HEADER1-TRACEDATA[2]-Pad18)
- DEBUG_HEADER1 pad 20: Net-(DEBUG_HEADER1-TRACEDATA[3]) -> unconnected-(DEBUG_HEADER1-TRACEDATA[3]-Pad20)
- H1 pad 23: +3.3VA -> +3.3V
- H1 pad 27: +3.3VA -> +3.3V
- H1 pad 31: Net-(DEBUG_HEADER1-TRACEDATA[1]) -> GND
- H1 pad 32: Net-(DEBUG_HEADER1-TRACEDATA[2]) -> GND
- H1 pad 33: Net-(DEBUG_HEADER1-TRACEDATA[3]) -> /FPGA/program_b
- H1 pad 34: Net-(DEBUG_HEADER1-TRACEDATA[0]) -> /FPGA/done
- H1 pad 35: Net-(DEBUG_HEADER1-TRACECLK) -> GND
- H1 pad 45: GND -> +3.3V
- H1 pad 46: unconnected-(H1-USB_VREGO-Pad46) -> +3.3V
- H1 pad 52: GND -> /microcontroller_unit/5V_IN
- J4 pad 1: Net-(U4B-IO_L5N_T0_AD13N_35) -> Net-(IC2-LED)
- J4 pad 2: Net-(U4B-IO_L6P_T0_35) -> Net-(D2-K)
- J4 pad 29: Net-(U4B-IO_L19N_T3_VREF_35) -> GND
- J4 pad 4: Net-(U4B-IO_L7P_T1_AD6P_35) -> +3.3V
- J6 pad 2: Net-(H1-PF10) -> Net-(J6-D-)
- J6 pad 3: Net-(H1-PF11) -> Net-(J6-D+)
- J6 pad S1: unconnected-(J6-SHIELD-PadS1) -> GND
- J6 pad S2: unconnected-(J6-SHIELD-PadS1) -> GND
- L1 pad 1: +1V8 -> Net-(JP3-A)
- L2 pad 2: +1V0 -> Net-(JP1-A)
- L3 pad 2: +3.3V -> Net-(JP2-A)
- R1 pad 1: +1V8 -> Net-(JP3-A)
- R17 pad 1: Net-(U4C-TMS_0) -> Net-(U4C-TCK_0)
- R3 pad 1: +1V0 -> Net-(JP1-A)
- R4 pad 2: Net-(U1-GND) -> GND
- R7 pad 1: +3.3V -> Net-(JP2-A)
- U1 pad 1: +1V0 -> Net-(JP1-A)
- U1 pad 5: Net-(U1-GND) -> GND
- U1 pad 8: Net-(U1-GND) -> GND
- U1 pad 9: Net-(U1-GND) -> GND
- U3 pad S1: unconnected-(U3-SHIELD-PadS1) -> GND
- U3 pad S2: unconnected-(U3-SHIELD-PadS1) -> GND
- U3 pad S3: unconnected-(U3-SHIELD-PadS1) -> GND
- U3 pad S4: unconnected-(U3-SHIELD-PadS1) -> GND
- U4 pad A13: GND -> unconnected-(U4A-IO_L7P_T1_AD2P_15-PadA13)
- U4 pad A14: GND -> unconnected-(U4A-IO_L7N_T1_AD2N_15-PadA14)
- U4 pad A15: GND -> unconnected-(U4A-IO_L9N_T1_DQS_AD3N_15-PadA15)
- U4 pad A3: GND -> unconnected-(U4B-IO_L4N_T0_35-PadA3)
- U4 pad A4: GND -> unconnected-(U4B-IO_L3N_T0_DQS_AD5N_35-PadA4)
- U4 pad A5: GND -> unconnected-(U4B-IO_L3P_T0_DQS_AD5P_35-PadA5)
- U4 pad A7: GND -> unconnected-(U4B-IO_L1N_T0_AD4N_35-PadA7)
- U4 pad B14: GND -> unconnected-(U4A-IO_L8N_T1_AD10N_15-PadB14)
- U4 pad B15: GND -> unconnected-(U4A-IO_L9P_T1_DQS_AD3P_15-PadB15)
- U4 pad B16: GND -> unconnected-(U4A-IO_L10N_T1_AD11N_15-PadB16)
- U4 pad B4: GND -> unconnected-(U4B-IO_L4P_T0_35-PadB4)
- U4 pad B5: GND -> unconnected-(U4B-IO_L2N_T0_AD12N_35-PadB5)
- U4 pad B6: GND -> unconnected-(U4B-IO_L2P_T0_AD12P_35-PadB6)
- U4 pad B7: GND -> unconnected-(U4B-IO_L1P_T0_AD4P_35-PadB7)
- U4 pad C14: GND -> unconnected-(U4A-IO_L8P_T1_AD10P_15-PadC14)
- U4 pad C16: GND -> unconnected-(U4A-IO_L10P_T1_AD11P_15-PadC16)
- U4 pad C3: Net-(U4B-IO_L7P_T1_AD6P_35) -> unconnected-(U4B-IO_L7P_T1_AD6P_35-PadC3)
- U4 pad C6: Net-(U4B-IO_L5N_T0_AD13N_35) -> unconnected-(U4B-IO_L5N_T0_AD13N_35-PadC6)
- U4 pad C7: GND -> unconnected-(U4B-IO_L5P_T0_AD13P_35-PadC7)
- U4 pad D6: Net-(U4B-IO_L6P_T0_35) -> unconnected-(U4B-IO_L6P_T0_35-PadD6)
- U4 pad D9: GND -> unconnected-(U4A-IO_L6N_T0_VREF_15-PadD9)
- U4 pad E6: GND -> unconnected-(U4B-IO_0_35-PadE6)
- U4 pad J4: Net-(U4B-IO_L19N_T3_VREF_35) -> unconnected-(U4B-IO_L19N_T3_VREF_35-PadJ4)
- U4 pad K13: GND -> unconnected-(U4A-IO_L5P_T0_D06_14-PadK13)
- U4 pad L13: GND -> unconnected-(U4A-IO_L5N_T0_D07_14-PadL13)
- U4 pad L14: GND -> unconnected-(U4A-IO_L4P_T0_D04_14-PadL14)
- U4 pad M12: GND -> unconnected-(U4A-IO_L6N_T0_D08_VREF_14-PadM12)
- U4 pad M14: GND -> unconnected-(U4A-IO_L4N_T0_D05_14-PadM14)
- U4 pad M15: GND -> unconnected-(U4A-IO_L3N_T0_DQS_EMCCLK_14-PadM15)
- U4 pad M16: GND -> unconnected-(U4A-IO_L7P_T1_D09_14-PadM16)
- U4 pad M6: GND -> unconnected-(U4A-IO_L19P_T3_A10_D26_14-PadM6)
- U4 pad N12: GND -> unconnected-(U4A-IO_L13N_T2_MRCC_14-PadN12)
- U4 pad N13: GND -> unconnected-(U4A-IO_L11P_T1_SRCC_14-PadN13)
- U4 pad N14: GND -> unconnected-(U4A-IO_L12P_T1_MRCC_14-PadN14)
- U4 pad N16: GND -> unconnected-(U4A-IO_L7N_T1_D10_14-PadN16)
- U4 pad N6: GND -> unconnected-(U4A-IO_L19N_T3_A09_D25_VREF_14-PadN6)
- U4 pad N9: GND -> unconnected-(U4A-IO_L18P_T2_A12_D28_14-PadN9)
- U4 pad P10: GND -> unconnected-(U4A-IO_L14P_T2_SRCC_14-PadP10)
- U4 pad P11: GND -> unconnected-(U4A-IO_L14N_T2_SRCC_14-PadP11)
- U4 pad P13: GND -> unconnected-(U4A-IO_L11N_T1_SRCC_14-PadP13)
- U4 pad P14: GND -> unconnected-(U4A-IO_L12N_T1_MRCC_14-PadP14)
- U4 pad P15: GND -> unconnected-(U4A-IO_L8P_T1_D11_14-PadP15)
- U4 pad P16: GND -> unconnected-(U4A-IO_L8N_T1_D12_14-PadP16)
- U4 pad P5: GND -> unconnected-(U4B-IO_L10P_T1_34-PadP5)
- U4 pad P6: GND -> unconnected-(U4A-IO_25_14-PadP6)
- U4 pad P8: GND -> unconnected-(U4A-IO_L20P_T3_A08_D24_14-PadP8)
- U4 pad P9: GND -> unconnected-(U4A-IO_L18N_T2_A11_D27_14-PadP9)
- U4 pad R10: GND -> unconnected-(U4A-IO_L17P_T2_A14_D30_14-PadR10)
- U4 pad R11: GND -> unconnected-(U4A-IO_L17N_T2_A13_D29_14-PadR11)
- U4 pad R12: GND -> unconnected-(U4A-IO_L15P_T2_DQS_RDWR_B_14-PadR12)
- U4 pad R13: GND -> unconnected-(U4A-IO_L16P_T2_CSI_B_14-PadR13)
- U4 pad R15: GND -> unconnected-(U4A-IO_L9P_T1_DQS_14-PadR15)
- U4 pad R16: GND -> unconnected-(U4A-IO_L9N_T1_DQS_D13_14-PadR16)
- U4 pad R5: GND -> unconnected-(U4A-IO_L23P_T3_A03_D19_14-PadR5)
- U4 pad R6: GND -> unconnected-(U4A-IO_L24P_T3_A01_D17_14-PadR6)
- U4 pad R7: GND -> unconnected-(U4A-IO_L24N_T3_A00_D16_14-PadR7)
- U4 pad R8: GND -> unconnected-(U4A-IO_L20N_T3_A07_D23_14-PadR8)
- U4 pad T10: GND -> unconnected-(U4A-IO_L22N_T3_A04_D20_14-PadT10)
- U4 pad T12: GND -> unconnected-(U4A-IO_L15N_T2_DQS_DOUT_CSO_B_14-PadT12)
- U4 pad T13: GND -> unconnected-(U4A-IO_L16N_T2_A15_D31_14-PadT13)
- U4 pad T14: GND -> unconnected-(U4A-IO_L10P_T1_D14_14-PadT14)
- U4 pad T15: GND -> unconnected-(U4A-IO_L10N_T1_D15_14-PadT15)
- U4 pad T3: GND -> unconnected-(U4B-IO_L9N_T1_DQS_34-PadT3)
- U4 pad T4: GND -> unconnected-(U4B-IO_L9P_T1_DQS_34-PadT4)
- U4 pad T5: GND -> unconnected-(U4A-IO_L23N_T3_A02_D18_14-PadT5)
- U4 pad T7: GND -> unconnected-(U4A-IO_L21P_T3_DQS_14-PadT7)
- U4 pad T8: GND -> unconnected-(U4A-IO_L21N_T3_DQS_A06_D22_14-PadT8)
- U4 pad T9: GND -> unconnected-(U4A-IO_L22P_T3_A05_D21_14-PadT9)
Routing:
- net /microcontroller_unit/5V_IN: track 0.00 -> 148.8 mm, vias 0 -> 4
- net Net-(U1-PG): track 0.00 -> 82.7 mm
- net GND: track 0.00 -> 69.0 mm, vias 0 -> 15
- net Net-(JP1-A): track 0.00 -> 51.3 mm, vias 0 -> 2
- net Net-(U2-VFB1): track 0.00 -> 38.4 mm, vias 0 -> 2
- net Net-(U1-VREG5): track 0.00 -> 25.8 mm
- net Net-(JP2-A): track 0.00 -> 24.2 mm
- net Net-(JP3-A): track 0.00 -> 23.1 mm
- net Net-(U2-EN2): track 0.00 -> 21.0 mm
- net Net-(U1-SW1): track 0.00 -> 16.5 mm
- net Net-(U2-SW1): track 0.00 -> 15.2 mm
- net Net-(U2-SW2): track 0.00 -> 14.5 mm
- net Net-(U1-VFB): track 0.00 -> 14.5 mm
- net Net-(U2-VBST2): track 0.00 -> 11.2 mm
- net Net-(U1-SS): track 0.00 -> 11.0 mm
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- added copper zone on In2.Cu, net +3.3V
- added copper zone on In1.Cu, net GND

Commit message: Work on PCB
Parts:
- moved C57 288.4 mm to (190.5, 60.0)
- moved C22 258.6 mm to (168.0, 115.5)
- moved C21 253.5 mm to (161.5, 128.5)
- moved C20 244.0 mm to (150.0, 138.3), turned to -90 degrees
- moved C23 211.4 mm to (113.8, 105.1)
- moved C94 138.9 mm to (180.5, 133.0), turned to 180 degrees
- moved R38 110.5 mm to (187.5, 127.5)
- moved R39 105.1 mm to (193.2, 127.5)
- moved C85 102.9 mm to (-4.27, 160.5)
- moved C86 102.9 mm to (-4.27, 163.5)
- moved C87 102.9 mm to (-4.27, 166.5)
- moved C88 102.9 mm to (0.54, 151.4)
- moved C89 102.9 mm to (0.54, 154.4)
- moved C90 102.9 mm to (0.54, 157.4)
- moved C91 102.9 mm to (0.54, 160.5)
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Routing:
- net GND: track 69.0 -> 309.5 mm, vias 15 -> 47
- net +3.3V: track 2.71 -> 149.6 mm, vias 1 -> 19
- net Net-(H1-PA1): track 0.00 -> 124.8 mm
- net Net-(H1-PA0): track 0.00 -> 110.2 mm
- net Net-(H1-PA3): track 0.00 -> 97.3 mm
- net Net-(H1-PD0): track 0.00 -> 94.1 mm
- net /microcontroller_unit/5V_IN: track 148.8 -> 238.7 mm, vias 4 -> 7
- net Net-(H1-PA2): track 0.00 -> 87.0 mm
- net Net-(H1-PD1): track 0.00 -> 83.0 mm
- net Net-(J5-Pad3): track 0.00 -> 50.2 mm
- net Net-(DEBUG_HEADER1-nRESET): track 0.00 -> 46.4 mm, vias 0 -> 2
- net Net-(J5-Pad1): track 0.00 -> 39.2 mm
- net Net-(H1-PF11): track 0.00 -> 39.0 mm, vias 0 -> 2
- net /FPGA/done: track 0.00 -> 37.5 mm, vias 0 -> 2
- net /FPGA/program_b: track 0.00 -> 34.8 mm, vias 0 -> 2
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
Commit message: Pcb
Parts:
- U4: footprint fpga:BGA256C100P16X16_1700X1700X155 -> fpga_real:BGA256C100P16X16_1700X1700X155
- moved C78 233.7 mm to (228.3, 44.0)
- moved C79 233.7 mm to (228.3, 47.0)
- moved C56 227.7 mm to (211.0, 43.8)
- moved C65 224.6 mm to (217.0, 47.0)
- moved C66 224.6 mm to (217.0, 50.1)
- moved C67 224.6 mm to (217.0, 53.1)
- moved C68 224.6 mm to (217.0, 56.1)
- moved C64 224.6 mm to (217.0, 44.0)
- moved C71 221.9 mm to (222.7, 44.0)
- moved C72 221.9 mm to (222.7, 47.0)
- moved C73 221.9 mm to (222.7, 50.0)
- moved C74 221.9 mm to (222.7, 53.0)
- moved C75 221.9 mm to (222.7, 56.0)
- moved C76 221.9 mm to (222.7, 59.0)
- moved C77 221.9 mm to (222.7, 62.0)
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Connections:
- J4 pad 35: Net-(U4B-IO_L22N_T3_35) -> unconnected-(J4-Pad35)
- J4 pad 36: Net-(U4B-IO_L23P_T3_35) -> unconnected-(J4-Pad36)
- J4 pad 37: Net-(U4B-IO_L23N_T3_35) -> unconnected-(J4-Pad37)
- J4 pad 38: Net-(U4B-IO_L24P_T3_35) -> unconnected-(J4-Pad38)
- J4 pad 39: Net-(U4B-IO_L24N_T3_35) -> unconnected-(J4-Pad39)
- J4 pad 40: Net-(U4B-IO_25_35) -> unconnected-(J4-Pad40)
- U4 pad J1: Net-(U4B-IO_L22N_T3_35) -> unconnected-(U4B-IO_L22N_T3_35-PadJ1)
- U4 pad K2: Net-(U4B-IO_L24N_T3_35) -> unconnected-(U4B-IO_L24N_T3_35-PadK2)
- U4 pad K3: Net-(U4B-IO_L24P_T3_35) -> unconnected-(U4B-IO_L24P_T3_35-PadK3)
- U4 pad K5: Net-(U4B-IO_25_35) -> unconnected-(U4B-IO_25_35-PadK5)
- U4 pad L2: Net-(U4B-IO_L23N_T3_35) -> unconnected-(U4B-IO_L23N_T3_35-PadL2)
- U4 pad L3: Net-(U4B-IO_L23P_T3_35) -> unconnected-(U4B-IO_L23P_T3_35-PadL3)
Routing:
- net GND: track 309.5 -> 667.8 mm, vias 47 -> 71
- net +3.3V: track 149.6 -> 388.4 mm, vias 19 -> 44
- net +1V0: track 0.00 -> 157.4 mm, vias 0 -> 2
- net +1V8: track 0.00 -> 94.9 mm, vias 0 -> 2
- net /FPGA/GREEN4: track 0.00 -> 92.4 mm, vias 0 -> 4
- net /FPGA/RED4: track 0.00 -> 83.2 mm, vias 0 -> 2
- net /FPGA/BLUE1: track 0.00 -> 80.9 mm, vias 0 -> 2
- net /FPGA/GREEN3: track 0.00 -> 75.9 mm, vias 0 -> 2
- net /FPGA/RED3: track 0.00 -> 75.8 mm, vias 0 -> 2
- net /FPGA/RED2: track 0.00 -> 74.9 mm, vias 0 -> 2
- net /FPGA/BLUE0: track 0.00 -> 73.9 mm, vias 0 -> 2
- net /FPGA/GREEN2: track 0.00 -> 72.7 mm, vias 0 -> 2
- net /FPGA/RED1: track 0.00 -> 72.7 mm, vias 0 -> 2
- net /FPGA/GREEN1: track 0.00 -> 70.3 mm, vias 0 -> 2
- net /FPGA/GREEN0: track 0.00 -> 69.9 mm, vias 0 -> 2
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
Commit message: hello
Parts:
- removed L2: 1.5u, Inductor_SMD:L_0805_2012Metric_Pad1.15x1.40mm_HandSolder
- moved C23 30.6 mm to (135.9, 89.4)
- moved Y2 30.6 mm to (136.2, 82.9)
- moved C48 26.5 mm to (229.9, 31.2)
- moved C49 26.5 mm to (230.0, 35.0)
- moved C50 26.5 mm to (230.0, 38.0)
- moved C51 26.5 mm to (230.0, 41.1)
- moved C52 26.5 mm to (230.0, 44.1)
- moved C53 26.5 mm to (230.0, 47.1)
- moved C54 26.5 mm to (230.0, 50.1)
- moved C55 26.5 mm to (230.0, 53.1)
- moved C56 26.5 mm to (236.0, 35.0)
- moved C58 26.5 mm to (236.0, 38.0)
- moved C59 26.5 mm to (236.0, 41.0)
- moved C60 26.5 mm to (236.0, 44.1)
- moved C61 26.5 mm to (236.0, 47.1)
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Routing:
- net GND: track 667.8 -> 319.7 mm, vias 71 -> 118
- net +3.3V: track 388.4 -> 168.2 mm, vias 44 -> 29
- net +1V0: track 157.4 -> 0.22 mm, vias 2 -> 0
- net +1V8: track 94.9 -> 0.06 mm, vias 2 -> 0
- net /FPGA/GREEN4: track 92.4 -> 0.00 mm, vias 4 -> 0
- net /FPGA/RED4: track 83.2 -> 0.00 mm, vias 2 -> 0
- net /FPGA/BLUE1: track 80.9 -> 0.00 mm, vias 2 -> 0
- net /FPGA/RED3: track 75.8 -> 0.00 mm, vias 2 -> 0
- net /FPGA/RED2: track 74.9 -> 0.00 mm, vias 2 -> 0
- net /FPGA/GREEN3: track 75.9 -> 1.36 mm, vias 2 -> 0
- net /FPGA/BLUE0: track 73.9 -> 0.00 mm, vias 2 -> 0
- net /FPGA/RED1: track 72.7 -> 0.00 mm, vias 2 -> 0
- net /FPGA/GREEN2: track 72.7 -> 1.24 mm, vias 2 -> 0
- net /FPGA/GREEN1: track 70.3 -> 0.00 mm, vias 2 -> 0
- net /FPGA/GREEN0: track 69.9 -> 0.00 mm, vias 2 -> 0
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- added copper zone on F.Cu, net GND

Commit message: pcb
Parts:
- moved C56 82.7 mm to (156.8, 59.2), turned to 90 degrees
- moved C48 80.9 mm to (156.6, 65.6), turned to 90 degrees
- moved C58 79.0 mm to (159.8, 59.2), turned to 90 degrees
- moved C49 75.8 mm to (160.5, 65.5), turned to 90 degrees
- moved C59 75.3 mm to (162.8, 59.2), turned to 90 degrees
- moved C57 73.9 mm to (138.3, 100.6)
- moved IC1 73.9 mm to (129.8, 97.4)
- moved R14 73.9 mm to (134.3, 106.6)
- moved R15 73.9 mm to (129.8, 106.6)
- moved R13 73.9 mm to (125.3, 106.6)
- moved C50 71.9 mm to (163.5, 65.5), turned to 90 degrees
- moved C60 71.7 mm to (165.8, 59.2), turned to 90 degrees
- moved C61 68.2 mm to (168.8, 59.2), turned to 90 degrees
- moved C51 68.0 mm to (166.5, 65.5), turned to 90 degrees
- moved C62 64.7 mm to (171.9, 59.2), turned to 90 degrees
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Routing:
- net +3.3V: track 168.2 -> 218.3 mm, vias 29 -> 63
- net GND: track 319.7 -> 369.2 mm, vias 118 -> 153
- net Net-(DEBUG_HEADER1-SWDCLK): track 8.46 -> 10.7 mm, vias 1 -> 0
- net (no net): vias 1 -> 0

Commit message: PCB
Parts:
- moved U4 5.55 mm to (149.5, 79.5)
Routing:
- net GND: track 369.2 -> 419.9 mm, vias 153 -> 164
- net +3.3V: track 218.3 -> 257.5 mm, vias 63 -> 71
- net +1V0: track 0.22 -> 11.4 mm, vias 0 -> 3
- net +1V8: track 0.06 -> 4.29 mm, vias 0 -> 3
- net Net-(U4B-IO_L13N_T2_MRCC_35): track 0.00 -> 1.06 mm, vias 0 -> 1
- net /FPGA/program_b: track 33.7 -> 34.4 mm, vias 2 -> 3
- net Net-(U4C-TCK_0): track 24.2 -> 24.9 mm, vias 0 -> 1
- net Net-(U4C-TDI_0): track 14.6 -> 15.3 mm, vias 0 -> 1
- net /FPGA/GPIO7: track 7.26 -> 7.97 mm, vias 0 -> 1
- net /FPGA/GPIO6: track 7.26 -> 7.97 mm, vias 0 -> 1
- net /FPGA/GPIO5: track 7.26 -> 7.97 mm, vias 0 -> 1
- net /FPGA/GPIO4: track 7.26 -> 7.97 mm, vias 0 -> 1
- net /FPGA/GPIO3: track 7.26 -> 7.97 mm, vias 0 -> 1
- net /FPGA/GPIO2: track 7.26 -> 7.97 mm, vias 0 -> 1
- net /FPGA/GPIO1: track 7.26 -> 7.97 mm, vias 0 -> 1
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
Commit message: work
Parts:
- moved C48 52.5 mm to (205.5, 46.4), turned to 180 degrees
- moved C49 50.5 mm to (205.5, 42.5), turned to 180 degrees
- moved C50 49.3 mm to (205.5, 39.5), turned to 180 degrees
- moved C51 48.6 mm to (205.5, 36.5), turned to 180 degrees
- moved C54 48.4 mm to (205.5, 27.5), turned to 180 degrees
- moved C52 48.1 mm to (205.5, 33.5), turned to 180 degrees
- moved C53 48.1 mm to (205.5, 30.5), turned to 180 degrees
- moved C56 44.2 mm to (199.1, 46.2), turned to 180 degrees
- moved C58 42.4 mm to (199.1, 43.2), turned to 180 degrees
- moved C59 41.0 mm to (199.1, 40.2), turned to 180 degrees
- moved C60 39.9 mm to (199.1, 37.2), turned to 180 degrees
- moved C63 39.4 mm to (199.1, 28.2), turned to 180 degrees
- moved C61 39.3 mm to (199.1, 34.2), turned to 180 degrees
- moved C62 39.1 mm to (199.1, 31.2), turned to 180 degrees
- moved C55 36.4 mm to (199.5, 51.2), turned to 0 degrees
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Routing:
- net /FPGA/GPIO5: track 7.97 -> 93.3 mm, vias 1 -> 2
- net /FPGA/GPIO4: track 7.97 -> 85.1 mm, vias 1 -> 2
- net /FPGA/GPIO6: track 7.97 -> 84.6 mm, vias 1 -> 2
- net /FPGA/GPIO3: track 7.97 -> 84.1 mm, vias 1 -> 2
- net /FPGA/GPIO2: track 7.97 -> 79.0 mm, vias 1 -> 2
- net /FPGA/GPIO1: track 7.97 -> 73.2 mm, vias 1 -> 2
- net /FPGA/GPIO0: track 7.97 -> 66.3 mm, vias 1 -> 2
- net /FPGA/GPIO7: track 7.97 -> 48.2 mm, vias 1 -> 2
- net /FPGA/MOSI: track 24.9 -> 60.3 mm, vias 3 -> 4
- net /FPGA/MISO: track 22.8 -> 53.9 mm, vias 3 -> 4
- net /FPGA/CLK: track 25.5 -> 55.1 mm, vias 3 -> 4
- net /FPGA/CS: track 26.6 -> 56.2 mm, vias 3 -> 4
- net /FPGA/program_b: track 34.4 -> 61.4 mm, vias 3 -> 2
- net /FPGA/done: track 37.1 -> 63.6 mm, vias 3 -> 2
- net Net-(DEBUG_HEADER1-SWDIO): track 12.3 -> 28.5 mm, vias 0 -> 2
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