File: PCB/mcu.kicad_sch (KiCad schematic)
At the start: 28 parts, among them J6 USB1130-15-A_REVA, SW1 SW_Push, SW2 SW_Push, SW3 SW_Push, SW4 SW_Push, U3 COM-09032, Y1 Crystal_GND24

Commit message: updates
Parts:
- added J3: FTS-102-02-F-DV-TR, 4pinHeader:FTS-102-YY-XX-DV-TR, symbol FTS-102-02-F-DV-TR:FTS-102-02-F-DV-TR
Connections:
- net GND: no longer H1.41 (PC8), H1.42 (PC9), H1.43 (PC10), H1.44 (PC11)
- new net: H1.41 (PC8), J3.1
- new net: H1.42 (PC9), J3.2
- new net: H1.43 (PC10), J3.4
- new net: H1.44 (PC11), J3.3
Changed lines of the file:
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@@
   (junction (at 88.9 158.75) (diameter 0) (color 0 0 0 0)
   )
-  (junction (at 121.92 87.63) (diameter 0) (color 0 0 0 0)
-  )
-  (junction (at 121.92 82.55) (diameter 0) (color 0 0 0 0)
-  )
   (junction (at 68.58 90.17) (diameter 0) (color 0 0 0 0)
   )
@@
   )
   (junction (at 49.53 60.96) (diameter 0) (color 0 0 0 0)
-  )
-  (junction (at 121.92 85.09) (diameter 0) (color 0 0 0 0)
   )
   (junction (at 68.58 102.87) (diameter 0) (color 0 0 0 0)
@@
     (stroke (width 0) (type default))
   )
+  (wire (pts (xy 121.92 85.09) (xy 160.02 85.09))
+    (stroke (width 0) (type default))
+  )
   (wire (pts (xy 88.9 146.05) (xy 88.9 158.75))
     (stroke (width 0) (type default))
@@
     (stroke (width 0) (type default))
   )
+  (wire (pts (xy 154.94 105.41) (xy 154.94 87.63))
+    (stroke (width 0) (type default))
+  )
   (wire (pts (xy 17.78 118.11) (xy 16.51 118.11))
     (stroke (width 0) (type default))
@@
     (stroke (width 0) (type default))
   )
+  (wire (pts (xy 152.4 90.17) (xy 121.92 90.17))
+    (stroke (width 0) (type default))
+  )
   (wire (pts (xy 121.92 80.01) (xy 128.27 80.01))
     (stroke (width 0) (type default))
@@
     (stroke (width 0) (type default))
   )
-  (wire (pts (xy 121.92 82.55) (xy 128.27 82.55))
-    (stroke (width 0) (type default))
-  )
   (wire (pts (xy 68.58 90.17) (xy 64.77 90.17))
     (stroke (width 0) (type default))
@@
     (stroke (width 0) (type default))
   )
-  (wire (pts (xy 121.92 82.55) (xy 121.92 85.09))
-    (stroke (width 0) (type default))
-  )
   (wire (pts (xy 45.72 72.39) (xy 68.58 72.39))
     (stroke (width 0) (type default))
   )
+  (wire (pts (xy 162.56 105.41) (xy 162.56 107.95))
+    (stroke (width 0) (type default))
+  )
   (wire (pts (xy 64.77 100.33) (xy 68.58 100.33))
     (stroke (width 0) (type default))
   )
+  (wire (pts (xy 154.94 87.63) (xy 121.92 87.63))
+    (stroke (width 0) (type default))
+  )
   (wire (pts (xy 27.94 83.82) (xy 33.02 83.82))
     (stroke (width 0) (type default))
@@
     (stroke (width 0) (type default))
   )
+  (wire (pts (xy 152.4 107.95) (xy 152.4 90.17))
+    (stroke (width 0) (type default))
+  )
   (wire (pts (xy 121.92 74.93) (xy 138.43 74.93))
     (stroke (width 0) (type default))
@@
     (stroke (width 0) (type default))
   )
+  (wire (pts (xy 160.02 105.41) (xy 154.94 105.41))
+    (stroke (width 0) (type default))
+  )
   (wire (pts (xy 204.47 46.99) (xy 114.3 46.99))
     (stroke (width 0) (type default))
@@
     (stroke (width 0) (type default))
   )
+  (wire (pts (xy 162.56 82.55) (xy 121.92 82.55))
+    (stroke (width 0) (type default))
+  )
   (wire (pts (xy 57.15 68.58) (xy 57.15 80.01))
     (stroke (width 0) (type default))
@@
     (stroke (width 0) (type default))
   )
-  (wire (pts (xy 121.92 87.63) (xy 121.92 90.17))
-    (stroke (width 0) (type default))
-  )
   (wire (pts (xy 139.7 60.96) (xy 149.86 60.96))
     (stroke (width 0) (type default))
@@
     (stroke (width 0) (type default))
   )
+  (wire (pts (xy 162.56 85.09) (xy 162.56 82.55))
+    (stroke (width 0) (type default))
+  )
   (wire (pts (xy 101.6 158.75) (xy 101.6 162.56))
     (stroke (width 0) (type default))
@@
     (stroke (width 0) (type default))
   )
+  (wire (pts (xy 162.56 107.95) (xy 152.4 107.95))
+    (stroke (width 0) (type default))
+  )
   (wire (pts (xy 101.6 52.07) (xy 104.14 52.07))
-    (stroke (width 0) (type default))
-  )
-  (wire (pts (xy 121.92 85.09) (xy 121.92 87.63))
     (stroke (width 0) (type default))
   )
@@
     )
   )
-  (symbol (lib_id "power:GND") (at 128.27 82.55 0) (unit 1)
-    (in_bom yes) (on_board yes) (dnp no)
-    (property "Reference" "#PWR064" (at 128.27 88.9 0)
-      (effects (font (size 1.27 1.27)) hide)
-    )
-    (property "Value" "GND" (at 130.81 86.36 0)
-      (effects (font (size 1.27 1.27)))
-    )
-    (property "Footprint" "" (at 128.27 82.55 0)
-      (effects (font (size 1.27 1.27)) hide)
-    )
-    (property "Datasheet" "" (at 128.27 82.55 0)
-      (effects (font (size 1.27 1.27)) hide)
-    )
-    (pin "1")
-    (instances
-      (project "PCB"
-        (path "/aa113cd6-c3ac-4890-9a84-1ea195994408/6d6ebb76-19de-41e4-9a7d-528f4e5c1c0f"
-          (reference "#PWR064") (unit 1)
-        )
-      )
-    )
-  )
   (symbol (lib_id "power:GND") (at 176.53 74.93 0) (unit 1)
     (in_bom yes) (on_board yes) (dnp no)
@@
         )
       )
+    )
+  )
+  (symbol (lib_id "FTS-102-02-F-DV-TR:FTS-102-02-F-DV-TR") (at 160.02 105.41 90) (unit 1)
+    (in_bom yes) (on_board yes) (dnp no) (fields_autoplaced)
+    (property "Reference" "J3" (at 166.37 93.98 90)
+      (effects (font (size 1.27 1.27)) (justify right))
+    )
+    (property "Value" "FTS-102-02-F-DV-TR" (at 166.37 96.52 90)
+      (effects (font (size 1.27 1.27)) (justify right))
+    )
+    (property "Footprint" "4pinHeader:FTS-102-YY-XX-DV-TR" (at 254.94 88.9 0)
+      (effects (font (size 1.27 1.27)) (justify left top) hide)
+    )
+    (property "Datasheet" "http://suddendocs.samtec.com/prints/fts-1xx-xx-xx-xx-xx-mkt.pdf" (at 354.94 88.9 0)
+      (effects (font (size 1.27 1.27)) (justify left top) hide)
+    )
+    (property "Height" "" (at 554.94 88.9 0)
+      (effects (font (size 1.27 1.27)) (justify left top) hide)
+    )
+    (property "Manufacturer_Name" "SAMTEC" (at 654.94 88.9 0)
+      (effects (font (size 1.27 1.27)) (justify left top) hide)
+    )
+    (property "Manufacturer_Part_Number" "FTS-102-02-F-DV-TR" (at 754.94 88.9 0)
+      (effects (font (size 1.27 1.27)) (justify left top) hide)
+    )
+    (property "Mouser Part Number" "200-FTS10202FDVTR" (at 854.94 88.9 0)
+      (effects (font (size 1.27 1.27)) (justify left top) hide)
+    )
+    (property "Mouser Price/Stock" "https://www.mouser.co.uk/ProductDetail/Samtec/FTS-102-02-F-DV-TR?qs=Cqqh%252BS766wn7Cg5YlIyggQ%3D%3D" (at 954.94 88.9 0)
+      (effects (font (size 1.27 1.27)) (justify left top) hide)
+    )
+    (property "Arrow Part Number" "FTS-102-02-F-DV-TR" (at 1054.94 88.9 0)
+      (effects (font (size 1.27 1.27)) (justify left top) hide)
+    )
+    (property "Arrow Price/Stock" "https://www.arrow.com/en/products/fts-102-02-f-dv-tr/samtec?region=nac" (at 1154.94 88.9 0)
+      (effects (font (size 1.27 1.27)) (justify left top) hide)
+    )
+    (pin "1")
+    (pin "2")
+    (pin "3")
+    (pin "4")
+    (instances
+      (project "PCB"
+        (path "/aa113cd6-c3ac-4890-9a84-1ea195994408/6d6ebb76-19de-41e4-9a7d-528f4e5c1c0f"
+          (reference "J3") (unit 1)
+        )
+      )
